File: src/resources/kicad/TROLL-SYSTEM/trollvalve.sch (KiCad schematic (older format))
At the start: 61 parts, among them K1 FINDER-32.21-x000, SW1 SW_DIP_x01, T2 CONN_01X01_MALE, T3 CONN_01X01_MALE, T4 CONN_01X01_MALE, U1 L78L05_SO8

Commit message: .
Parts:
- added U?: CARLINGSW_L, symbol trollvalve:CARLINGSW_L
Changed lines of the file:
@@
 	-1   0    0    1
 $EndComp
+$Comp
+L trollvalve:CARLINGSW_L U?
+U 1 1 5E23D65F
+P 8050 5300
+F 0 "U?" H 8475 6265 50  0000 C CNN
+F 1 "CARLINGSW_L" H 8475 6174 50  0000 C CNN
+F 2 "" H 8250 5150 50  0001 C CNN
+F 3 "" H 8250 5150 50  0001 C CNN
+	1    8050 5300
+	1    0    0    -1
+$EndComp
 $EndSCHEMATC
