File: src/resources/kicad/DC-HELM-DISTRIBUTION-CABINET/helm-wiring.sch (KiCad schematic (older format))
At the start: 330 parts, among them P106 114, P107 119, P108 120, P109 121, P11 01, P110 122, P111 123, P112 124, P113 125, P114 126, P115 127, P116 128, P117 129, P118 130, P119 131, P12 02, P120 132, P121 133, P122 134, P123 135, P124 136, P125 137, P126 138, P127 139, P128 140, P129 141, P13 03, P14 04, P18 08, P19 09, P20 10, P21 13, P22 14, P23 15, P26 04, P27 05, P28 25, P29 01, P30 02, P31 03, P32 04, P33 05, P34 06, P35 07, P36 08, P37 09, P38 10, P39 11, P40 12, P41 13, P42 01, P43 02, P44 03, P47 06, P49 01, P50 03, P51 04, P52 05, P53 06, P54 07, P55 08, P56 09, P57 10, P58 11, P59 13, P60 14, P61 15, P62 17, P63 18, P64 19, P65 20, P66 21, P67 22, P68 23

Commit message: .
Parts:
- removed P106: 114, symbol helm-wiring-rescue:CONN_02X01-beatrice-helm-wiring-rescue-helm-wiring-rescue
- removed P107: 119, symbol helm-wiring-rescue:CONN_02X01-beatrice-helm-wiring-rescue-helm-wiring-rescue
- removed P108: 120, symbol helm-wiring-rescue:CONN_02X01-beatrice-helm-wiring-rescue-helm-wiring-rescue
- removed P109: 121, symbol helm-wiring-rescue:CONN_02X01-beatrice-helm-wiring-rescue-helm-wiring-rescue
- removed P110: 122, symbol helm-wiring-rescue:CONN_02X01-beatrice-helm-wiring-rescue-helm-wiring-rescue
- removed P111: 123, symbol helm-wiring-rescue:CONN_02X01-beatrice-helm-wiring-rescue-helm-wiring-rescue
- removed P112: 124, symbol helm-wiring-rescue:CONN_02X01-beatrice-helm-wiring-rescue-helm-wiring-rescue
- removed P113: 125, symbol helm-wiring-rescue:CONN_02X01-beatrice-helm-wiring-rescue-helm-wiring-rescue
- removed P114: 126, symbol helm-wiring-rescue:CONN_02X01-beatrice-helm-wiring-rescue-helm-wiring-rescue
- removed P115: 127, symbol helm-wiring-rescue:CONN_02X01-beatrice-helm-wiring-rescue-helm-wiring-rescue
- removed P116: 128, symbol helm-wiring-rescue:CONN_02X01-beatrice-helm-wiring-rescue-helm-wiring-rescue
- removed P117: 129, symbol helm-wiring-rescue:CONN_02X01-beatrice-helm-wiring-rescue-helm-wiring-rescue
- removed P118: 130, symbol helm-wiring-rescue:CONN_02X01-beatrice-helm-wiring-rescue-helm-wiring-rescue
- removed P119: 131, symbol helm-wiring-rescue:CONN_02X01-beatrice-helm-wiring-rescue-helm-wiring-rescue
- removed P120: 132, symbol helm-wiring-rescue:CONN_02X01-beatrice-helm-wiring-rescue-helm-wiring-rescue
- removed P121: 133, symbol helm-wiring-rescue:CONN_02X01-beatrice-helm-wiring-rescue-helm-wiring-rescue
- removed P122: 134, symbol helm-wiring-rescue:CONN_02X01-beatrice-helm-wiring-rescue-helm-wiring-rescue
- removed P123: 135, symbol helm-wiring-rescue:CONN_02X01-beatrice-helm-wiring-rescue-helm-wiring-rescue
- removed P124: 136, symbol helm-wiring-rescue:CONN_02X01-beatrice-helm-wiring-rescue-helm-wiring-rescue
- removed P125: 137, symbol helm-wiring-rescue:CONN_02X01-beatrice-helm-wiring-rescue-helm-wiring-rescue
- removed P126: 138, symbol helm-wiring-rescue:CONN_02X01-beatrice-helm-wiring-rescue-helm-wiring-rescue
- removed P127: 139, symbol helm-wiring-rescue:CONN_02X01-beatrice-helm-wiring-rescue-helm-wiring-rescue
- removed P128: 140, symbol helm-wiring-rescue:CONN_02X01-beatrice-helm-wiring-rescue-helm-wiring-rescue
- removed P129: 141, symbol helm-wiring-rescue:CONN_02X01-beatrice-helm-wiring-rescue-helm-wiring-rescue
- removed P?: 111, symbol helm-wiring-rescue:CONN_02X01-beatrice-helm-wiring-rescue-helm-wiring-rescue
- removed P?: 112, symbol helm-wiring-rescue:CONN_02X01-beatrice-helm-wiring-rescue-helm-wiring-rescue
- removed P?: 113, symbol helm-wiring-rescue:CONN_02X01-beatrice-helm-wiring-rescue-helm-wiring-rescue
- removed P?: 115, symbol helm-wiring-rescue:CONN_02X01-beatrice-helm-wiring-rescue-helm-wiring-rescue
- removed P?: 116, symbol helm-wiring-rescue:CONN_02X01-beatrice-helm-wiring-rescue-helm-wiring-rescue
- removed P?: 117, symbol helm-wiring-rescue:CONN_02X01-beatrice-helm-wiring-rescue-helm-wiring-rescue
- removed P?: 118, symbol helm-wiring-rescue:CONN_02X01-beatrice-helm-wiring-rescue-helm-wiring-rescue
- removed P?: 142, symbol helm-wiring-rescue:CONN_02X01-beatrice-helm-wiring-rescue-helm-wiring-rescue
- removed P? (x2): 143, symbol helm-wiring-rescue:CONN_02X01-beatrice-helm-wiring-rescue-helm-wiring-rescue
- removed P? (x2): 45, symbol helm-wiring-rescue:CONN_02X01-beatrice-helm-wiring-rescue-helm-wiring-rescue
- removed P? (x2): 44, symbol helm-wiring-rescue:CONN_02X01-beatrice-helm-wiring-rescue-helm-wiring-rescue
- removed P?: 42, symbol helm-wiring-rescue:CONN_02X01-beatrice-helm-wiring-rescue-helm-wiring-rescue
- removed P?: 40, symbol helm-wiring-rescue:CONN_02X01-beatrice-helm-wiring-rescue-helm-wiring-rescue
- removed P?: 41, symbol helm-wiring-rescue:CONN_02X01-beatrice-helm-wiring-rescue-helm-wiring-rescue
- removed P?: 43, symbol helm-wiring-rescue:CONN_02X01-beatrice-helm-wiring-rescue-helm-wiring-rescue
- removed P?: 46, symbol helm-wiring-rescue:CONN_02X01-beatrice-helm-wiring-rescue-helm-wiring-rescue
- added P? (x2): 01, symbol helm-wiring-rescue:CONN_02X01-beatrice-helm-wiring-rescue-helm-wiring-rescue-he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
- added P? (x2): 04, symbol helm-wiring-rescue:CONN_02X01-beatrice-helm-wiring-rescue-helm-wiring-rescue-he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
- added P? (x2): 05, symbol helm-wiring-rescue:CONN_02X01-beatrice-helm-wiring-rescue-helm-wiring-rescue-he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
- added P? (x2): 06, symbol helm-wiring-rescue:CONN_02X01-beatrice-helm-wiring-rescue-helm-wiring-rescue-he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
- added P? (x2): 08, symbol helm-wiring-rescue:CONN_02X01-beatrice-helm-wiring-rescue-helm-wiring-rescue-he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
- added P? (x2): 07, symbol helm-wiring-rescue:CONN_02X01-beatrice-helm-wiring-rescue-helm-wiring-rescue-he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
- added P? (x2): 03, symbol helm-wiring-rescue:CONN_02X01-beatrice-helm-wiring-rescue-helm-wiring-rescue-he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
- added P? (x2): 02, symbol helm-wiring-rescue:CONN_02X01-beatrice-helm-wiring-rescue-helm-wiring-rescue-he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
- added P?: 25, symbol helm-wiring-rescue:CONN_02X01-beatrice-helm-wiring-rescue-helm-wiring-rescue-he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
- added P?: 09, symbol helm-wiring-rescue:CONN_02X01-beatrice-helm-wiring-rescue-helm-wiring-rescue-he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
- added P?: 18, symbol helm-wiring-rescue:CONN_02X01-beatrice-helm-wiring-rescue-helm-wiring-rescue-he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
- added P?: 19, symbol helm-wiring-rescue:CONN_02X01-beatrice-helm-wiring-rescue-helm-wiring-rescue-he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
- added P?: 17, symbol helm-wiring-rescue:CONN_02X01-beatrice-helm-wiring-rescue-helm-wiring-rescue-he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
- added P?: 10, symbol helm-wiring-rescue:CONN_02X01-beatrice-helm-wiring-rescue-helm-wiring-rescue-he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
- added P?: 11, symbol helm-wiring-rescue:CONN_02X01-beatrice-helm-wiring-rescue-helm-wiring-rescue-he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
- added P?: 14, symbol helm-wiring-rescue:CONN_02X01-beatrice-helm-wiring-rescue-helm-wiring-rescue-he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
- added P?: 15, symbol helm-wiring-rescue:CONN_02X01-beatrice-helm-wiring-rescue-helm-wiring-rescue-he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
- added P?: 20, symbol helm-wiring-rescue:CONN_02X01-beatrice-helm-wiring-rescue-helm-wiring-rescue-he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
- added P?: 21, symbol helm-wiring-rescue:CONN_02X01-beatrice-helm-wiring-rescue-helm-wiring-rescue-he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
- added P?: 22, symbol helm-wiring-rescue:CONN_02X01-beatrice-helm-wiring-rescue-helm-wiring-rescue-he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
- added P?: 23, symbol helm-wiring-rescue:CONN_02X01-beatrice-helm-wiring-rescue-helm-wiring-rescue-he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
- added P?: 24, symbol helm-wiring-rescue:CONN_02X01-beatrice-helm-wiring-rescue-helm-wiring-rescue-he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
- added P?: 16, symbol helm-wiring-rescue:CONN_02X01-beatrice-helm-wiring-rescue-helm-wiring-rescue-he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
- added P?: 12, symbol helm-wiring-rescue:CONN_02X01-beatrice-helm-wiring-rescue-helm-wiring-rescue-he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
- added P?: 13, symbol helm-wiring-rescue:CONN_02X01-beatrice-helm-wiring-rescue-helm-wiring-rescue-he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
- added P?: 26, symbol helm-wiring-rescue:CONN_02X01-beatrice-helm-wiring-rescue-helm-wiring-rescue-he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
- P11, P12, P13, P14, P18, P19, P20, P21, P22, P23, P26, P27, P28, P29, P30, P31, P32, P33, P34, P35, P36, P37, P38, P39, P40, P41, P42, P43, P44, P47, P49, P50, P51, P52, P53, P54, P55, P56, P57, P58, P59, P60, P61, P62, P63, P64, P65, P66, P67, P68, P? (x56): symbol helm-wiring-rescue:CONN_02X01-beatrice-helm-wiring-rescue-helm-wiring-rescue -> helm-wiring-rescue:CONN_02X01-beatrice-helm-wiring-rescue-helm-wiring-rescue-helm-wiring-rescue
- RL?: value VHF -> SPUD
Connections:
- net labels added: AIS_NOTRANSMIT, NMEA_CONTROLLER_5A, SPUD_RLY, TROLL_SW_ON
- net labels removed: AIS_TRANSCEIVER_NOTRANSMIT, HP_DCKLTS_ON, HP_HYDRLC_EN
- wire segments 342 -> 350
Other:
- note removed: "EQUIPMENT CONNECTIONS"
- note removed: "EXTERNAL\nINPUTS"
- note removed: "OR 2.5"
- note removed: "OR/BK 1.5"
- note removed: "OR/BK 2.5"
- note removed: "RD/BK 1.0"
- note removed: "RD/BK 1.5"
- note removed: "RD/BK 2.5"
