File: src/resources/kicad/schematics/dc-helm.sch (KiCad schematic (older format))
At the start: 321 parts, among them P11 01, P12 02, P13 03, P14 04, P18 08, P19 09, P20 10, P21 13, P22 14, P23 15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

Commit message: Refactor
Parts:
- P11, P12, P13, P14, P18, P19, P20, P21, P22, P23, P26, P27, P28, P29, P30, P31, P32, P33, P34, P35, P36, P37, P38, P39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: symbol helm-wiring-rescue:CONN_02X01-beatrice-helm-wiring-rescue-helm-wiring-rescue-helm-wiring-rescue -> beatrice:DIN_RAIL_TERMINAL
