File: src/resources/kicad/schematics/dc-master-cabin.sch (KiCad schematic (older format))
At the start: 38 parts

Commit message: Refactor
Parts:
- (spare), F0, F09, F1, F10, F11, F12, F13, F14, F15, F16, F2, F3, F4, F5: symbol FUSE -> MC-DISTRIBUTION-CABINET-rescue:FUSE
- F? (x17): symbol FUSE_TERMINAL -> MC-DISTRIBUTION-CABINET-rescue:FUSE_TERMINAL
- SP?: symbol DEPTH/LOG -> MC-DISTRIBUTION-CABINET-rescue:DEPTH_LOG
- U? (x2): symbol NMEA_3478 -> MC-DISTRIBUTION-CABINET-rescue:NMEA_3478
- U?: symbol NMEA_FPM100 -> MC-DISTRIBUTION-CABINET-rescue:NMEA_FPM100
Changed lines of the file:
@@
-EESchema Schematic File Version 2
-LIBS:power
-LIBS:device
-LIBS:transistors
-LIBS:conn
-LIBS:linear
-LIBS:regul
-LIBS:74xx
-LIBS:cmos4000
-LIBS:adc-dac
-LIBS:memory
-LIBS:xilinx
-LIBS:microcontrollers
-LIBS:dsp
-LIBS:microchip
-LIBS:analog_switches
-LIBS:motorola
-LIBS:texas
-LIBS:intel
-LIBS:audio
-LIBS:interface
-LIBS:digital-audio
-LIBS:philips
-LIBS:display
-LIBS:cypress
-LIBS:siliconi
-LIBS:opto
-LIBS:atmel
-LIBS:contrib
-LIBS:valves
-LIBS:MC-DISTRIBUTION-CABINET-cache
-EELAYER 25 0
+EESchema Schematic File Version 4
+EELAYER 30 0
 EELAYER END
 $Descr A4 11693 8268
@@
 $EndDescr
 $Comp
-L NMEA_3478 U?
+L MC-DISTRIBUTION-CABINET-rescue:NMEA_3478 U?
 U 1 1 581F0063
 P 1050 5450
@@
 $EndComp
 $Comp
-L NMEA_3478 U?
+L MC-DISTRIBUTION-CABINET-rescue:NMEA_3478 U?
 U 1 1 581F01EE
 P 7640 5450
@@
 $EndComp
 $Comp
-L FUSE F1
+L MC-DISTRIBUTION-CABINET-rescue:FUSE F1
 U 1 1 581F05F2
 P 4100 3240
@@
 	4100 2360 4100 3240
 $Comp
-L FUSE F2
+L MC-DISTRIBUTION-CABINET-rescue:FUSE F2
 U 1 1 581F0A8E
 P 4500 3240
@@
 	4500 2360 4500 3240
 $Comp
-L FUSE F4
+L MC-DISTRIBUTION-CABINET-rescue:FUSE F4
 U 1 1 581F0CF2
 P 5300 3240
@@
 	5300 2360 5300 3240
 $Comp
-L FUSE F3
+L MC-DISTRIBUTION-CABINET-rescue:FUSE F3
 U 1 1 581F0EC3
 P 4900 3240
@@
 	4900 2360 4900 3240
 $Comp
-L FUSE F5
+L MC-DISTRIBUTION-CABINET-rescue:FUSE F5
 U 1 1 581F0F3D
 P 5700 3240
@@
 	5700 2360 5700 3240
 $Comp
-L FUSE (spare)
+L MC-DISTRIBUTION-CABINET-rescue:FUSE (spare)
 U 1 1 581F1038
 P 6100 3240
@@
 	6100 2360 6100 3240
 $Comp
-L FUSE (spare)
+L MC-DISTRIBUTION-CABINET-rescue:FUSE (spare)
 U 1 1 581F10C8
 P 6500 3240
@@
 	6500 2360 6500 3240
 $Comp
-L FUSE (spare)
+L MC-DISTRIBUTION-CABINET-rescue:FUSE (spare)
 U 1 1 581F117F
 P 6900 3240
@@
 Wire Wire Line
 	5300 3740 5300 3940
-Connection ~ 5300 3940
 Wire Wire Line
 	4900 3740 4900 3940
-Connection ~ 4900 3940
 Wire Wire Line
 	4500 3740 4500 3940
-Connection ~ 4500 3940
 Wire Wire Line
 	6100 3940 6100 3740
-Connection ~ 5700 3940
 Wire Wire Line
 	6500 3940 6500 3740
-Connection ~ 6100 3940
 Wire Wire Line
 	6900 3940 6900 3740
-Connection ~ 6500 3940
-$Comp
-L FUSE F09
+$Comp
+L MC-DISTRIBUTION-CABINET-rescue:FUSE F09
 U 1 1 581F2ADC
 P 7420 3240
@@
 Wire Wire Line
 	7420 3940 7420 3740
-Connection ~ 6900 3940
-$Comp
-L FUSE F10
+$Comp
+L MC-DISTRIBUTION-CABINET-rescue:FUSE F10
 U 1 1 581F3769
 P 7820 3240
@@
 	7820 2360 7820 3240
 $Comp
-L FUSE F11
+L MC-DISTRIBUTION-CABINET-rescue:FUSE F11
 U 1 1 581F3770
 P 8220 3240
@@
 	8220 2360 8220 3240
 $Comp
-L FUSE F13
+L MC-DISTRIBUTION-CABINET-rescue:FUSE F13
 U 1 1 581F3777
 P 9020 3240
@@
 	9020 2360 9020 3240
 $Comp
-L FUSE F12
+L MC-DISTRIBUTION-CABINET-rescue:FUSE F12
 U 1 1 581F377E
 P 8620 3240
@@
 	8620 2360 8620 3240
 $Comp
-L FUSE F14
+L MC-DISTRIBUTION-CABINET-rescue:FUSE F14
 U 1 1 581F3785
 P 9420 3240
@@
 	9420 2360 9420 3240
 $Comp
-L FUSE F15
+L MC-DISTRIBUTION-CABINET-rescue:FUSE F15
 U 1 1 581F378C
 P 9820 3240
@@
 	9820 2360 9820 3240
 $Comp
-L FUSE F16
+L MC-DISTRIBUTION-CABINET-rescue:FUSE F16
 U 1 1 581F3793
 P 10220 3240
@@
 Wire Wire Line
 	7820 3940 7820 3740
-Connection ~ 7420 3940
 Wire Wire Line
 	8220 3940 8220 3740
-Connection ~ 7820 3940
 Wire Wire Line
 	8620 3940 8620 3740
-Connection ~ 8220 3940
 Wire Wire Line
 	9020 3940 9020 3740
-Connection ~ 8620 3940
 Wire Wire Line
 	9420 3940 9420 3740
 Wire Wire Line
 	9820 3940 9820 3740
-Connection ~ 9420 3940
 Wire Wire Line
 	10220 3940 10220 3740
-Connection ~ 9820 3940
-Connection ~ 9020 3940
 Wire Notes Line
 	7660 1300 7660 1340
@@
 	11040 1420 11040 2610
 $Comp
-L DEPTH/LOG SP?
+L MC-DISTRIBUTION-CABINET-rescue:DEPTH_LOG SP?
 U 1 1 581FAB4F
 P 15150 2950
@@
 NMEA MALE TERMINATOR
 $Comp
-L NMEA_FPM100 U?
+L MC-DISTRIBUTION-CABINET-rescue:NMEA_FPM100 U?
 U 1 1 581FC32D
 P 2130 2360
@@
 Wire Bus Line
 	2290 1120 4100 1120
-Connection ~ 4100 3940
 Text Notes 660  3920 0    60   ~ 0
 +24VDC 60A (25mm)\nFROM DC LINKBOX
@@
 TO BW PUMP (4mm)
 $Comp
-L FUSE F0
+L MC-DISTRIBUTION-CABINET-rescue:FUSE F0
 U 1 1 58205E71
 P 3730 3240
@@
 Wire Wire Line
 	3730 3740 3730 3940
-Connection ~ 3730 3940
 Wire Wire Line
 	3730 3240 3730 3200
@@
 TO SPUD POLE (4mm)
 $Comp
-L FUSE_TERMINAL F?
+L MC-DISTRIBUTION-CABINET-rescue:FUSE_TERMINAL F?
 U 1 1 5820B91C
 P 1060 4360
@@
 	1050 5450 1050 4810
 $Comp
-L FUSE_TERMINAL F?
+L MC-DISTRIBUTION-CABINET-rescue:FUSE_TERMINAL F?
 U 1 1 5820BDF5
 P 1260 4360
@@
 	1350 5450 1350 4810
 $Comp
-L FUSE_TERMINAL F?
+L MC-DISTRIBUTION-CABINET-rescue:FUSE_TERMINAL F?
 U 1 1 5820BE95
 P 1460 4360
@@
 	1750 5450 1750 4810
 $Comp
-L FUSE_TERMINAL F?
+L MC-DISTRIBUTION-CABINET-rescue:FUSE_TERMINAL F?
 U 1 1 5820BF67
 P 1660 4360
@@
 	2150 5450 2150 4810
 $Comp
-L FUSE_TERMINAL F?
+L MC-DISTRIBUTION-CABINET-rescue:FUSE_TERMINAL F?
 U 1 1 5820C01B
 P 1860 4360
@@
 	2550 5450 2550 4810
 $Comp
-L FUSE_TERMINAL F?
+L MC-DISTRIBUTION-CABINET-rescue:FUSE_TERMINAL F?
 U 1 1 5820C0C7
 P 2060 4360
@@
 	2950 5450 2950 4810
 $Comp
-L FUSE_TERMINAL F?
+L MC-DISTRIBUTION-CABINET-rescue:FUSE_TERMINAL F?
 U 1 1 5820C1D1
 P 2260 4360
@@
 	3350 5450 3350 4810
 $Comp
-L FUSE_TERMINAL F?
+L MC-DISTRIBUTION-CABINET-rescue:FUSE_TERMINAL F?
 U 1 1 5820C2B9
 P 2460 4360
@@
 	3750 5450 3750 4810
 $Comp
-L FUSE_TERMINAL F?
+L MC-DISTRIBUTION-CABINET-rescue:FUSE_TERMINAL F?
 U 1 1 58249E47
 P 2660 4360
@@
 $EndComp
 $Comp
-L FUSE_TERMINAL F?
+L MC-DISTRIBUTION-CABINET-rescue:FUSE_TERMINAL F?
 U 1 1 58249E4D
 P 2860 4360
@@
 $EndComp
 $Comp
-L FUSE_TERMINAL F?
+L MC-DISTRIBUTION-CABINET-rescue:FUSE_TERMINAL F?
 U 1 1 58249E53
 P 3060 4360
@@
 $EndComp
 $Comp
-L FUSE_TERMINAL F?
+L MC-DISTRIBUTION-CABINET-rescue:FUSE_TERMINAL F?
 U 1 1 58249E59
 P 3260 4360
@@
 $EndComp
 $Comp
-L FUSE_TERMINAL F?
+L MC-DISTRIBUTION-CABINET-rescue:FUSE_TERMINAL F?
 U 1 1 58249E5F
 P 3460 4360
@@
 $EndComp
 $Comp
-L FUSE_TERMINAL F?
+L MC-DISTRIBUTION-CABINET-rescue:FUSE_TERMINAL F?
 U 1 1 58249E65
 P 3660 4360
@@
 $EndComp
 $Comp
-L FUSE_TERMINAL F?
+L MC-DISTRIBUTION-CABINET-rescue:FUSE_TERMINAL F?
 U 1 1 58249E6B
 P 3860 4360
@@
 $EndComp
 $Comp
-L FUSE_TERMINAL F?
+L MC-DISTRIBUTION-CABINET-rescue:FUSE_TERMINAL F?
 U 1 1 58249E71
 P 4060 4360
@@
 $EndComp
 $Comp
-L FUSE_TERMINAL F?
+L MC-DISTRIBUTION-CABINET-rescue:FUSE_TERMINAL F?
 U 1 1 58249EB9
 P 4260 4360
