File: src/resources/kicad/schematics/troll-system-overview.sch (KiCad schematic (older format))
At the start: 61 parts, among them K1 FINDER-32.21-x000, T2 CONN_01X01_MALE, T3 CONN_01X01_MALE, T4 CONN_01X01_MALE, U1 L78L05_SO8

Commit message: Refactor
Parts:
- added T? (x6): Conn_01x01_Male, symbol Connector:Conn_01x01_Male
- 1.5A, 2A, 500mA, 5A: symbol trollvalve-rescue:Fuse-trollvalve-rescue -> Device:Fuse
- C1, C2, C3, C4, C5, C6, C7, C8, T2, T3, T4, T? (x8): value CONN_01X01_MALE -> Conn_01x01_Male; symbol trollvalve-rescue:CONN_01X01_MALE-trollvalve-rescue -> Connector:Conn_01x01_Male
- J? (x20): symbol trollvalve-rescue:CONN_01X01_FEMALE-trollvalve-rescue -> Connector:Conn_01x01_Female
- J? (x7): value CONN_01X01_FEMALE -> Conn_01x01_Female; symbol trollvalve-rescue:CONN_01X01_FEMALE-trollvalve-rescue -> Connector:Conn_01x01_Female
- M?: symbol trollvalve-rescue:Stepper_Motor_bipolar-trollvalve-rescue -> Motor:Stepper_Motor_bipolar
- SL?: symbol trollvalve-rescue:Solenoid-trollvalve -> beatrice:Solenoid
- SW?: symbol trollvalve-rescue:SW_Push_SPDT-trollvalve-rescue -> Switch:SW_SPDT
- U?: symbol trollvalve-rescue:POLOLU_TIC_T500-trollvalve -> beatrice:POLOLU_TIC_T500
Connections:
- wire segments 111 -> 110
