File: src/resources/kicad/schematics/main-engine-wiring-cabinet.sch (KiCad schematic (older format))
At the start: 12 parts, among them K1 MAIN ENGINE START, K2 SHAFT LUBE PUMP, U1 POLOLU_TIC_T500

Commit message: Refactor
Parts:
- U1: symbol dc-main-engine-connection-box-rescue:POLOLU_TIC_T500-trollvalve -> beatrice:POLOLU_TIC_T500
Changed lines of the file:
@@
 Connection ~ 2450 6200
 $Comp
-L dc-main-engine-connection-box-rescue:POLOLU_TIC_T500-trollvalve U1
+L beatrice:POLOLU_TIC_T500 U1
 U 1 1 5E31D2A1
 P 8500 4200
