File: src/resources/kicad/schematics/helm-wiring-cabinet.sch (KiCad schematic (older format))
At the start: 324 parts, among them P11 01, P12 02, P13 03, P14 04, P18 08, P19 09, P20 10, P21 13, P22 14, P23 15, P26 04, P27 05, P28 25, P29 01, P30 02, P31 03, P32 04, P33 05, P34 06, P35 07, P36 08, P37 09, P38 10, P39 11, P40 12, P41 13, P42 01, P43 02, P44 03, P47 06, P49 01, P50 03, P51 04, P52 05, P53 06, P54 07, P55 08, P56 09, P57 10, P58 11, P59 13, P60 14, P61 15, P62 17, P63 18, P64 19, P65 20, P66 21, P67 22, P68 23

Commit message: Revised wiring
Parts:
- added K?: COURTESY_LIGHTS, Relay_THT:Relay_SPST_Finder_32.21-x300, symbol Relay:FINDER-32.21-x000
- added P?: 01, symbol beatrice:DIN_RAIL_TERMINAL
- added P?: 04, symbol beatrice:DIN_RAIL_TERMINAL
- added P?: 05, symbol beatrice:DIN_RAIL_TERMINAL
- added P?: 06, symbol beatrice:DIN_RAIL_TERMINAL
- added P? (x2): 08, symbol beatrice:DIN_RAIL_TERMINAL
- added P?: 07, symbol beatrice:DIN_RAIL_TERMINAL
- added P?: 03, symbol beatrice:DIN_RAIL_TERMINAL
- added P?: 02, symbol beatrice:DIN_RAIL_TERMINAL
- added P?: 41, symbol beatrice:DIN_RAIL_TERMINAL
- added P?: 42, symbol beatrice:DIN_RAIL_TERMINAL
- added P?: 43, symbol beatrice:DIN_RAIL_TERMINAL
- added P?: 44, symbol beatrice:DIN_RAIL_TERMINAL
- added P?: 09, symbol beatrice:DIN_RAIL_TERMINAL
- added P?: 10, symbol beatrice:DIN_RAIL_TERMINAL
Connections:
- net labels added: BLUEBOARD_+-24VDC_5A, CALL_FOR_PROPANE_GAS, HP_NITELT_+24VDC, HP_NITELT_ON_POS1, HP_NITELT_ON_POS2, HP_WRKLT_+24VDC, HP_WRKLT_[DECK]-ON, HP_WRKLT_[STROBE]_ON, NMEA_VOLTAGE_REFERENCE_5A, SP_ALERT_LED, SP_DN_LED, SP_DOWN, SP_ENABLE_SWITCH-P1, SP_ENABLE_SWITCH-P2, SP_ENABLE_SWITCH_+24VDC, SP_GND, SP_ISOL_BLK, SP_ISOL_RED, SP_IS_DOWN, SP_IS_UP, SP_POLE_+24VDC, SP_POLE_GND, SP_UP, SP_UPDN_SWITCH_+24VDC, SP_UPDN_SWITCH_DN, SP_UPDN_SWITCH_UP, SP_UP_LED
- net labels removed: BLUEBOARD_+/-24VDC_5A, HP_NITELT_ON, HP_WRKLT_ON, PROPANE_GAS_ON, TROLL_SW_ON, WIPER_+24VDC_10A, WIPER_MODE_+24VDC_10A
- wire segments 330 -> 318
