File: resources/kicad/schematics/dc/helm/helm.kicad_sch (KiCad schematic)
At the start: 371 parts, among them J1 01, J10 10, J100 33, J101 34, J102 35, J103 36, J104 37, J105 38, J106 39, J107 29, J108 01, J109 02, J11 11, J110 03, J111 04, J112 05, J113 06, J114 40, J115 01, J116 02, J117 03, J118 04, J119 05, J12 12, J120 06, J121 07, J122 08, J123 09, J124 10, J125 11, J126 12, J127 13, J128 14, J129 15, J13 13, J130 16, J131 17, J132 18, J133 19, J134 20, J135 21, J136 22, J137 23, J138 24, J139 25, J14 14, J140 26, J141 27, J142 28, J143 07, J144 08, J145 09, J146 02, J147 05, J148 03, J149 01, J15 15, J150 02, J151 05, J152 06, J153 09, J154 07, J155 09, J156 15, J157 14, J158 16, J159 20, J16 16, J160 21, J161 08, J162 25, J163 38, J164 39, J165 13, J166 32, J167 11, J168 40, J169 09, J17 17, J170 41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

Commit message: Updates
Parts:
- removed F1: 500mA, symbol Device:Fuse
- removed F2: 5A, symbol Device:Fuse
- removed J10, J124, J40, J77: 10, symbol Beatrice:Conn_02x01_24VDC
- removed J100: 33, symbol Beatrice:Conn_02x01_24VDC
- removed J101: 34, symbol Beatrice:Conn_02x01_24VDC
- removed J102: 35, symbol Beatrice:Conn_02x01_24VDC
- removed J103: 36, symbol Beatrice:Conn_02x01_24VDC
- removed J104: 37, symbol Beatrice:Conn_02x01_24VDC
- removed J105: 38, symbol Beatrice:Conn_02x01_24VDC
- removed J106: 39, symbol Beatrice:Conn_02x01_24VDC
- removed J107, J29, J96: 29, symbol Beatrice:Conn_02x01_24VDC
- removed J108, J115, J298, J31, J62, J68: 01, symbol Beatrice:Conn_02x01_24VDC
- removed J109, J116, J299, J32, J63, J69: 02, symbol Beatrice:Conn_02x01_24VDC
- removed J11, J125, J41, J78: 11, symbol Beatrice:Conn_02x01_24VDC
- removed J110, J117, J300, J33, J64, J70: 03, symbol Beatrice:Conn_02x01_24VDC
- removed J111, J118, J34, J65, J71: 04, symbol Beatrice:Conn_02x01_24VDC
- removed J112, J119, J35, J5, J66, J72: 05, symbol Beatrice:Conn_02x01_24VDC
- removed J113, J120, J36, J6, J67, J73: 06, symbol Beatrice:Conn_02x01_24VDC
- removed J114: 40, symbol Beatrice:Conn_02x01_24VDC
- removed J12, J126, J42, J61, J79: 12, symbol Beatrice:Conn_02x01_24VDC
- removed J121, J143, J37, J7, J74: 07, symbol Beatrice:Conn_02x01_24VDC
- removed J122, J144, J38, J75, J8: 08, symbol Beatrice:Conn_02x01_24VDC
- removed J123, J145, J39, J76, J9: 09, symbol Beatrice:Conn_02x01_24VDC
- removed J127, J13, J199, J43, J80: 13, symbol Beatrice:Conn_02x01_24VDC
- removed J128, J14, J44, J81: 14, symbol Beatrice:Conn_02x01_24VDC
- removed J129, J15, J45, J82: 15, symbol Beatrice:Conn_02x01_24VDC
- removed J130, J16, J46, J83: 16, symbol Beatrice:Conn_02x01_24VDC
- removed J131, J17, J47, J84: 17, symbol Beatrice:Conn_02x01_24VDC
- removed J132, J18, J48, J85: 18, symbol Beatrice:Conn_02x01_24VDC
- removed J133, J19, J86: 19, symbol Beatrice:Conn_02x01_24VDC
- removed J134, J20, J87: 20, symbol Beatrice:Conn_02x01_24VDC
- removed J135, J21, J88: 21, symbol Beatrice:Conn_02x01_24VDC
- removed J136, J22, J89: 22, symbol Beatrice:Conn_02x01_24VDC
- removed J137, J23, J90: 23, symbol Beatrice:Conn_02x01_24VDC
- removed J138, J24, J91: 24, symbol Beatrice:Conn_02x01_24VDC
- removed J139, J25, J92: 25, symbol Beatrice:Conn_02x01_24VDC
- removed J140, J26, J93: 26, symbol Beatrice:Conn_02x01_24VDC
- removed J141, J27, J94: 27, symbol Beatrice:Conn_02x01_24VDC
- removed J142, J28, J95: 28, symbol Beatrice:Conn_02x01_24VDC
- removed J154: 07, symbol Beatrice:Conn_02x01_4MM2_BLUE
- removed J180: 54, symbol Beatrice:Conn_02x01_24VDC
- removed J186, J98: 31, symbol Beatrice:Conn_02x01_24VDC
- removed J227: 01, symbol Beatrice:Conn_02x01_4MM2_BLUE
- removed J229: 02, symbol Beatrice:Conn_02x01_4MM2_BLUE
- removed J231, J271, J273, J274, J275, J277, J278, J279, J280, J281: 10, symbol Beatrice:Conn_02x01_4MM2_BLUE
- removed J233: 03, symbol Beatrice:Conn_02x01_4MM2_GREY
- removed J272: 04, symbol Beatrice:Conn_02x01_4MM2_GREY
- removed J292: 05, symbol Beatrice:Conn_02x01_4MM2_GREY
- removed J297: 06, symbol Beatrice:Conn_02x01_4MM2_GREY
- removed J30, J97: 30, symbol Beatrice:Conn_02x01_24VDC
- removed J311, J312: 08, symbol Beatrice:Conn_02x01_4MM2_BLUE
- removed J49: 01, symbol Beatrice:Conn_03x01
- removed J50: 02, symbol Beatrice:Conn_03x01
- removed J51: 03, symbol Beatrice:Conn_03x01
- removed J52: 04, symbol Beatrice:Conn_03x01
- removed J53: 05, symbol Beatrice:Conn_03x01
- removed J54: 06, symbol Beatrice:Conn_03x01
- removed J55: 07, symbol Beatrice:Conn_03x01
- removed J56: 08, symbol Beatrice:Conn_03x01
- removed J57: 09, symbol Beatrice:Conn_03x01
- removed J58: 10, symbol Beatrice:Conn_03x01
- removed J59: 11, symbol Beatrice:Conn_03x01
- removed J99: 32, symbol Beatrice:Conn_02x01_24VDC
- added D1, D2: D_Small, symbol Device:D_Small
- added J180: 20, symbol Beatrice:Conn_02x01_4MM2_BLUE
- added J313: 08, symbol Beatrice:Conn_02x01_4MM2_BLUE
- added J314: 09, symbol Beatrice:Conn_02x01_4MM2_BLUE
- J1: value 01 -> 20
- J155, J302: value 09 -> 10
- J194: value 06 -> 07
- J2: value 02 -> 42
- J220: value 12 -> 14
- J221: value 08 -> 21
- J223: value 13 -> 15
- J224: value 14 -> 16
- J226: value 20 -> 23
- J228: value 10 -> 11
- J230: value 09 -> 03
- J232: value 11 -> 12
- J234: value 15 -> 17
- J235: value 16 -> 18
- J236: value 17 -> 19
- J237: value 18 -> 13
- J238: value 19 -> 22
- J250: value 21 -> 24
- J251: value 22 -> 25
- J276: value 09 -> 08
- J282: value 09 -> 04
- J283: value 15 -> 14
- J284: value 16 -> 15
- J289: value 09 -> 05
- J290: value 09 -> 06
- J296: value 09 -> 07
- J3: value 03 -> 53
- J303: value 09 -> 11
- J304: value 09 -> 12
- J308: value 09 -> 13
- J4: value 04 -> 53
Connections:
- net DECK_LIGHTS(WHEELHOUSE)_+ is gone; now on net SPUD_ISOLATOR_+/-: J221. (Pin_2)
- net HP.ENG.IGN is gone; now on net IGN.75: J159. (Pin_2)
- net HP.ENG.IGN.TRL.SBY is gone; now on net IGN.75.TRL.SBY: J309. (Pin_2)
- net HP.ENG.RPM.ALM is gone; now on net TSR.COIL: J310. (Pin_2)
- net HP.SW12.T04 is gone; now on net WL.COIL: J307. (Pin_2)
- net HP.SW16.T01 is gone; now on net WIPER_ON: J243. (Pin_2)
- net HP.SW16.T04 is gone; now on net WIPER_MODE: J191. (Pin_2)
- net HP.SW19.T03 is gone; now on net HP.F5.1.4.EBP.SBY: J261. (Pin_2)
- net HP.SW19.T04 is gone; now on net HPA.3: J263. (Pin_2)
- net HP.SW20.T03 is gone; now on net HP.F5.1.5.MCB.SBY: J266. (Pin_2)
- net HP.SW20.T04 is gone; now on net HPA.4: J267. (Pin_2)
- net HP.SW21.T03 is gone; now on net NMEA_1.02: J181. (Pin_2)
- net HP.SW21.T04 is gone; now on net NMEA_1.03: J182. (Pin_2)
- net HP.SW22.T03 is gone; now on net NMEA_1.04: J244. (Pin_2)
- net HP.SW22.T04 is gone; now on net NMEA_1.05: J245. (Pin_2)
- net HP.SW33.T04 is gone; now on net WIFI_ON: J247. (Pin_2)
- net MAIN_ISOLATOR_NO (ACTIVE LOW) is gone; now on net NIGHT_LIGHT_ON: J2. (Pin_2)
- net MAIN_ISOLATOR_RELAY is gone; now on net NIGHT_LIGHT_ON: J2. (Pin_2)
- net NMEA_0.09 is gone; now on net NMEA_1.10: J3. (Pin_2)
- net NMEA_1.01 is gone; now on net NMEA_INTERFACE2_+: U4. (CANBUS)
- net PA_CHANNEL_02 is gone; now on net MC.BILGE_SENSOR_FLOAT_SW_NO: J259. (Pin_2)
- net PA_CHANNEL_03 is gone; now on net HPA.3: J263. (Pin_2), J264. (Pin_2)
- net TSR.ENG.IGN is gone; now on net IGN.75.TRL.SBY: J309. (Pin_2)
- net WORK_LIGHT_ON is gone; now on net WORK_LIGHT_+: J251. (Pin_2)
- net F9.1.1: no longer J1. (Pin_2)
- net F9.1.9.WL: now also J251. (Pin_2)
- net HPA.2: now also J259. (Pin_2)
- net HPA.4: now also J268. (Pin_2)
- net NMEA_1.10: no longer J174. (Pin_2), J178. (Pin_2), J209. (Pin_2)
- net NMEA_ETH.IO5P: now also J239. (Pin_2)
- net HP.F5.1.4.EBP.SBY: now reaches J261. (Pin_2)
- net HP.F5.1.4.EBP.SBY: no longer J262. (Pin_2)
- net HP.F9.2.8.THR.OP1: now reaches J4. (Pin_2)
- net HP.F9.2.8.THR.OP1: now also J3. (Pin_2)
- net IGN.75.TRL.SBY: now reaches K3.11
- net IGN.75.TRL.SBY: now also K3.A2
- net HP.F5.1.5.MCB.SBY: now reaches J266. (Pin_2)
- net HP.F5.1.5.MCB.SBY: no longer J269. (Pin_2)
- net HP.F9.2.8.THR.ACT: now reaches J178. (Pin_2)
- net BC.MAIN_ISOLATOR_SOLENOID_BLACK renamed MAIN_ISOLATOR_SOLENOID_BLACK
- net BC.MAIN_ISOLATOR_SOLENOID_RED renamed MAIN_ISOLATOR_SOLENOID_RED
- net DECK_LIGHTS(WHEELHOUSE) renamed SPUD_ISOLATOR_+/-
- net SPUD_ISOLATOR_+/-: now also J180. (Pin_2)
- net DP.24VDC_BUSBAR renamed IGN.75
- net IGN.75: now also U4. (CANBUS)
- removed net DP.ANCHOR_LIGHT_SW_NO: J3. (Pin_2), J4. (Pin_2)
- net ENG.IGN.ALM renamed IGN.75.TRL.SBY.A
- net IGN.75.TRL.SBY.A: now also J313. (Pin_2)
- net ENG.IGN.SBY renamed IGN.75.TRL.SBY.B
- net IGN.75.TRL.SBY.B: now also U4. (CANBUS), J314. (Pin_2)
- net HP.SW19.T02 renamed HP.F5.1.4
- net HP.SW20.T02 renamed HP.F5.1.5
- net HP.SW31,T03 renamed SOLENOID R
- net SOLENOID R: now also D2.2 (A)
- net HP.SW31.T02 renamed SOLENOID L
- net SOLENOID L: now also D1.2 (A)
- removed net NMEA_1.16: J159. (Pin_2), U4. (CANBUS)
- removed net PA_CHANNEL_04: J267. (Pin_2), J268. (Pin_2)
- new net: J261. (Pin_2), J262. (Pin_2)
- new net: D1.1 (K), D2.1 (K), J178. (Pin_2)
- new net: J266. (Pin_2), J269. (Pin_2)
- new net F9.1.8.SPUD.A: J180. (Pin_2)
- new net F9.1.8.SPUD.B: J221. (Pin_2)
- new net HP.F5.1.4.EBP.OP1: J263. (Pin_2)
- new net HP.F5.1.5.MCB.OP1: J267. (Pin_2)
- new net HP.F9.1.2.ERV.OP1: J182. (Pin_2)
- new net HP.F9.1.2.ERV.SBY: J181. (Pin_2)
- new net HP.F9.1.2.MBV.OP1: J245. (Pin_2)
- new net HP.F9.1.2.MBV.SBY: J244. (Pin_2)
- new net HP.F9.1.7.WIF.OP1: J247. (Pin_2)
- new net HP.F9.2.1.WNL.OP1: J2. (Pin_2)
- new net HP.F9.2.7.WPR.CFG: J191. (Pin_2)
- new net HP.F9.2.7.WPR.OP1: J243. (Pin_2)
- new net HP.F9.2.8.THR.LFT: J174. (Pin_2), J209. (Pin_2)
- new net HP.GND.RPM.ALM: J310. (Pin_2)
- new net HP.GND.WKL.OP1: J307. (Pin_2)
- new net HP.IGN.75: J159. (Pin_2)
- new net HP.IGN.75.TRL.SBY: J309. (Pin_2)
- new net HP.IGN.75.TRL.SBY.A: J313. (Pin_2)
- new net HP.IGN.75.TRL.SBY.B: J314. (Pin_2)
Other:
- note added: "DIM13-2DIN is a two-rail dimmer providing a 5W PWM positive supply and a 5W PWM ground sink. An SSD timer relay extends both rails with an intermittent characteristic."
- note added: "The Courtesy Light Relay (CLR) switches power to the wheelhouse courtesy lights and is operated by physical switches at the helm and domestic panels and by an NMEA modulated remote relay."
- note removed: "A 2-rail dimmer (DIM13-2DIN) provides a 5W PWM positive supply and a 5W PWM ground sink. An SSD timer relay extends both rails with an intermittent characteristic."
- note removed: "AIS"
- note removed: "AIS TRANSCEIVER (EMTRAK)"
- note removed: "ALARM MODULE CHANNEL USAGE 01 - ER BILGE LEVEL HIGH 02 - MC BILGE LEVEL HIGH 03 - ER BILGE PUMP RUNNING 04 - MC BILGE PUMP RUNNING 05 - WASTE DISCHARGE PUMP RUNNING 06 - SPUD ALARM 07 08 - BATTERY VOLTAGE LOW 09 - FIRE ALARM ACTIVE 10 - INTRUDER ALARM ACTIVE"
- note removed: "ANCHOR"
- note removed: "ANCHOR LIGHT (WHEELHOUSE)"
- note removed: "BLUE BOARD"
- note removed: "COOLING"
- note removed: "COURTESY LIGHTS"
- note removed: "DECK LIGHTS (WHEELHOUSE)"
- note removed: "DECK WASH"
- note removed: "DEHUMIDIFIER"
- note removed: "ENGINE"
- note removed: "FORE LOCKER"
- note removed: "GAS ISOLATOR"
- note removed: "GENERATOR REMOTE START"
- note removed: "GENERATOR SENSOR"
- note removed: "HEATING"
- note removed: "HEATING PROGRAMMER"
- note removed: "HELM ISOLATOR"
- note removed: "HORN"
- note removed: "HOT WATER"
- note removed: "IMMERSION HEATER 1KW"
- note removed: "IMMERSION HEATER 2KW"
- note removed: "MAIN ISOLATOR RREVERSING RELAY"
- note removed: "MAST"
- note removed: "NMEA"
- note removed: "NMEA BUS 0"
- note removed: "NMEA BUS 1"
- note removed: "NON-FOLLOW-UP"
- note removed: "RADAR"
- note removed: "SEARCHLIGHT"
- note removed: "SPUD POLE"
- note removed: "SPUDPOLE"
- note removed: "THRUSTERS"
- note removed: "TROLL"
- note removed: "TROLL SWITCH"
- note removed: "TROLL SYSTEM"
- note removed: "The Courtesy Light Relay (CL) switches power to the wheelhouse courtesy lights and is operated by physical switches at the helm and domestic panels and by an NMEA modulated remote relay."
- note removed: "VENTILATION (MB)"
- note removed: "VENTILATOR (ER)"
- note removed: "VHF"
- note removed: "WHEELHOUSE LIGHTS"
- note removed: "WIFI"
- note removed: "WIPER"
- note removed: "WORK LIGHT"

Commit message: Add helm panel lighting on-off feature.
Parts:
- added J5: 02, symbol Beatrice:Conn_02x01_24VDC
Connections:
- net F5.1.7: no longer RL9.A1, U2. (SUPPLY)
- new net: J261. (Pin_2), J262. (Pin_2)
- new net: J266. (Pin_2), J269. (Pin_2)
- new net F5.1.7.HPD.SBY: J5. (Pin_2), RL9.A1, U2. (SUPPLY)
- new net HP.F5.1.7.HPD.SBY: J5. (Pin_2)

Commit message: Tidy up
Parts:
- added J6: 15, symbol Beatrice:Conn_02x01_4MM2_BLUE
- added J7: 16, symbol Beatrice:Conn_02x01_4MM2_BLUE
- J225: value 15 -> 17
- J248: value 16 -> 18
- J249: value 17 -> 19
Connections:
- net F9.3.3: now also J6. (Pin_2)
- net F9.3.5: now also J7. (Pin_2)
- new net: J261. (Pin_2), J262. (Pin_2)
- new net: J266. (Pin_2), J269. (Pin_2)
- new net HP.F9.3.3: J6. (Pin_2)
- new net HP.F9.3.5: J7. (Pin_2)

Commit message: Reformat switch diagram
Connections:
- new net: J261. (Pin_2), J262. (Pin_2)
- new net: J266. (Pin_2), J269. (Pin_2)
Changed lines of the file:
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@@
 	)
 	(symbol
-		(lib_name "Beatrice:Conn_02x01_24VDC")
 		(lib_id "Beatrice:Conn_02x01_24VDC")
 		(at 236.22 350.52 90)
@@
 	)
 	(symbol
-		(lib_name "Beatrice:Conn_02x01_4MM2_GREY")
 		(lib_id "Beatrice:Conn_02x01_4MM2_GREY")
 		(at 373.38 350.52 90)
@@
 	)
 	(symbol
-		(lib_name "Beatrice:Conn_02x01_4MM2_GREY")
 		(lib_id "Beatrice:Conn_02x01_4MM2_GREY")
 		(at 365.76 350.52 90)
@@
 	)
 	(symbol
-		(lib_name "Beatrice:Conn_02x01_24VDC")
 		(lib_id "Beatrice:Conn_02x01_24VDC")
 		(at 292.1 350.52 90)
@@
 	)
 	(symbol
-		(lib_name "Beatrice:Conn_02x01_24VDC")
 		(lib_id "Beatrice:Conn_02x01_24VDC")
 		(at 269.24 350.52 90)
@@
 	)
 	(symbol
-		(lib_name "Beatrice:Conn_02x01_24VDC")
 		(lib_id "Beatrice:Conn_02x01_24VDC")
 		(at 226.06 350.52 90)
@@
 	)
 	(symbol
-		(lib_name "Beatrice:Conn_02x01_24VDC")
 		(lib_id "Beatrice:Conn_02x01_24VDC")
 		(at 287.02 350.52 90)
@@
 	)
 	(symbol
-		(lib_name "Beatrice:Conn_02x01_24VDC")
 		(lib_id "Beatrice:Conn_02x01_24VDC")
 		(at 243.84 350.52 90)
@@
 	)
 	(symbol
-		(lib_name "Beatrice:Conn_02x01_24VDC")
 		(lib_id "Beatrice:Conn_02x01_24VDC")
 		(at 271.78 350.52 90)
@@
 	)
 	(symbol
-		(lib_name "Beatrice:Conn_02x01_24VDC")
 		(lib_id "Beatrice:Conn_02x01_24VDC")
 		(at 284.48 350.52 90)
@@
 	)
 	(symbol
-		(lib_name "Beatrice:Conn_02x01_24VDC")
 		(lib_id "Beatrice:Conn_02x01_24VDC")
 		(at 289.56 350.52 90)
@@
 	)
 	(symbol
-		(lib_name "Beatrice:Conn_02x01_24VDC")
 		(lib_id "Beatrice:Conn_02x01_24VDC")
 		(at 228.6 350.52 90)
@@
 	)
 	(symbol
-		(lib_name "Beatrice:Conn_02x01_24VDC")
 		(lib_id "Beatrice:Conn_02x01_24VDC")
 		(at 266.7 350.52 90)
@@
 	)
 	(symbol
-		(lib_name "Beatrice:Conn_02x01_24VDC")
 		(lib_id "Beatrice:Conn_02x01_24VDC")
 		(at 368.3 350.52 90)
@@
 	)
 	(symbol
-		(lib_name "Beatrice:Conn_02x01_24VDC")
 		(lib_id "Beatrice:Conn_02x01_24VDC")
 		(at 274.32 350.52 90)
@@
 	)
 	(symbol
-		(lib_name "Beatrice:Conn_02x01_24VDC")
 		(lib_id "Beatrice:Conn_02x01_24VDC")
 		(at 281.94 350.52 90)
@@
 	)
 	(symbol
-		(lib_name "Beatrice:Conn_02x01_24VDC")
 		(lib_id "Beatrice:Conn_02x01_24VDC")
 		(at 370.84 350.52 90)
@@
 	)
 	(symbol
-		(lib_name "Beatrice:Conn_02x01_24VDC")
 		(lib_id "Beatrice:Conn_02x01_24VDC")
 		(at 213.36 350.52 90)
@@
 	)
 	(symbol
-		(lib_name "Beatrice:Conn_02x01_4MM2_GREY")
 		(lib_id "Beatrice:Conn_02x01_4MM2_GREY")
 		(at 378.46 350.52 90)

Commit message: Update helm.kicad_sch
Parts:
- added J10, J8, J9: 06, symbol Beatrice:Conn_02x01_24VDC
Connections:
- net HP.F9.2.8.THR.LFT: no longer J209. (Pin_2)
- net HP.F9.2.8.THR.OP1: no longer J4. (Pin_2)
- net VHF_+: no longer J226. (Pin_2)
- net HP.F9.2.8.THR.OP2: now reaches J4. (Pin_2)
- new net: J261. (Pin_2), J262. (Pin_2)
- new net: J266. (Pin_2), J269. (Pin_2)
- new net AUTOPILOT_L: J9. (Pin_2)
- new net AUTOPILOT_LR: J8. (Pin_2)
- new net AUTOPILOT_R: J10. (Pin_2)
- new net HP.AUTOPILOT_L: J9. (Pin_2)
- new net HP.AUTOPILOT_LR: J8. (Pin_2)
- new net HP.AUTOPILOT_R: J10. (Pin_2)
- new net HP.F9.2.8.THR.RGT: J209. (Pin_2)
- new net HP.VHF_+: J226. (Pin_2)

Commit message: Add wire colors / sizes
Connections:
- new net: J261. (Pin_2), J262. (Pin_2)
- new net: J266. (Pin_2), J269. (Pin_2)
Changed lines of the file:
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@@
 	)
 	(symbol
-		(lib_name "Beatrice:Conn_02x01_24VDC")
 		(lib_id "Beatrice:Conn_02x01_24VDC")
 		(at 243.84 350.52 90)
@@
 	)
 	(symbol
-		(lib_name "Beatrice:Conn_02x01_4MM2_GREY")
 		(lib_id "Beatrice:Conn_02x01_4MM2_GREY")
 		(at 381 350.52 90)
@@
 	)
 	(symbol
-		(lib_name "Beatrice:Conn_02x01_4MM2_GREY")
 		(lib_id "Beatrice:Conn_02x01_4MM2_GREY")
 		(at 373.38 350.52 90)
@@
 	)
 	(symbol
-		(lib_name "Beatrice:Conn_02x01_24VDC")
 		(lib_id "Beatrice:Conn_02x01_24VDC")
 		(at 299.72 350.52 90)
@@
 	)
 	(symbol
-		(lib_name "Beatrice:Conn_02x01_24VDC")
 		(lib_id "Beatrice:Conn_02x01_24VDC")
 		(at 276.86 350.52 90)
@@
 	)
 	(symbol
-		(lib_name "Beatrice:Conn_02x01_24VDC")
 		(lib_id "Beatrice:Conn_02x01_24VDC")
 		(at 233.68 350.52 90)
@@
 	)
 	(symbol
-		(lib_name "Beatrice:Conn_02x01_24VDC")
 		(lib_id "Beatrice:Conn_02x01_24VDC")
 		(at 294.64 350.52 90)
@@
 	)
 	(symbol
-		(lib_name "Beatrice:Conn_02x01_24VDC")
 		(lib_id "Beatrice:Conn_02x01_24VDC")
 		(at 251.46 350.52 90)
@@
 	)
 	(symbol
-		(lib_name "Beatrice:Conn_02x01_24VDC")
 		(lib_id "Beatrice:Conn_02x01_24VDC")
 		(at 279.4 350.52 90)
@@
 	)
 	(symbol
-		(lib_name "Beatrice:Conn_02x01_24VDC")
 		(lib_id "Beatrice:Conn_02x01_24VDC")
 		(at 292.1 350.52 90)
@@
 	)
 	(symbol
-		(lib_name "Beatrice:Conn_02x01_24VDC")
 		(lib_id "Beatrice:Conn_02x01_24VDC")
 		(at 297.18 350.52 90)
@@
 	)
 	(symbol
-		(lib_name "Beatrice:Conn_02x01_24VDC")
 		(lib_id "Beatrice:Conn_02x01_24VDC")
 		(at 236.22 350.52 90)
@@
 	)
 	(symbol
-		(lib_name "Beatrice:Conn_02x01_24VDC")
 		(lib_id "Beatrice:Conn_02x01_24VDC")
 		(at 274.32 350.52 90)
@@
 	)
 	(symbol
-		(lib_name "Beatrice:Conn_02x01_24VDC")
 		(lib_id "Beatrice:Conn_02x01_24VDC")
 		(at 375.92 350.52 90)
@@
 	)
 	(symbol
-		(lib_name "Beatrice:Conn_02x01_24VDC")
 		(lib_id "Beatrice:Conn_02x01_24VDC")
 		(at 281.94 350.52 90)
@@
 	)
 	(symbol
-		(lib_name "Beatrice:Conn_02x01_24VDC")
 		(lib_id "Beatrice:Conn_02x01_24VDC")
 		(at 289.56 350.52 90)
@@
 	)
 	(symbol
-		(lib_name "Beatrice:Conn_02x01_24VDC")
 		(lib_id "Beatrice:Conn_02x01_24VDC")
 		(at 378.46 350.52 90)
@@
 	)
 	(symbol
-		(lib_name "Beatrice:Conn_02x01_24VDC")
 		(lib_id "Beatrice:Conn_02x01_24VDC")
 		(at 213.36 350.52 90)
@@
 	)
 	(symbol
-		(lib_name "Beatrice:Conn_02x01_4MM2_GREY")
 		(lib_id "Beatrice:Conn_02x01_4MM2_GREY")
 		(at 386.08 350.52 90)

Commit message: Tweak
Parts:
- removed J252: 06, symbol Beatrice:Conn_02x01_4MM2_BLUE
- removed J253: 07, symbol Beatrice:Conn_02x01_4MM2_BLUE
- removed RL9: MAIN ISOLATOR RELAY (MI), symbol Relay:FINDER-40.52
- added K2: FINDER-32.21-x000, Relay_THT:Relay_SPDT_Finder_32.21-x000, symbol Relay:FINDER-32.21-x000
- J285: value 02 -> 03
- J286: value 03 -> 04
- J287: value 04 -> 05
- J288: value 05 -> 06
Connections:
- net F5.1.7.HPD.PWM is gone; now on net HPD.INC: U2. (SUPPLY)
- net F5.1.7.HPD.SBY: now also K2.A1
- net GND: now also K2.A2
- net GND.HPD.PWM: now also K2.11
- net GND.HPD.PWM.INT: now also K2.14
- new net: J261. (Pin_2), J262. (Pin_2)
- new net: J266. (Pin_2), J269. (Pin_2)
Other:
- note added: "DIM13-2DIN is a two-rail dimmer providing a 5W PWM positive supply (unused) and a 5W PWM ground sink. An SSD timer relay extends the sink rail with an intermittent characteristic."
- note removed: "DIM13-2DIN is a two-rail dimmer providing a 5W PWM positive supply and a 5W PWM ground sink. An SSD timer relay extends both rails with an intermittent characteristic."

Commit message: Many tweaks
Parts:
- removed J149: 01, symbol Beatrice:Conn_02x01_4MM2_GREY
- removed J150: 02, symbol Beatrice:Conn_02x01_24VDC
- removed J153: 09, symbol Beatrice:Conn_02x01_24VDC
- removed J156: 15, symbol Beatrice:Conn_02x01_24VDC
- removed J157: 14, symbol Beatrice:Conn_02x01_24VDC
- removed J163: 38, symbol Beatrice:Conn_02x01_24VDC
- removed J168: 40, symbol Beatrice:Conn_02x01_24VDC
- removed J169, J314: 09, symbol Beatrice:Conn_02x01_4MM2_BLUE
- removed J173: 49, symbol Beatrice:Conn_02x01_24VDC
- removed J180: 20, symbol Beatrice:Conn_02x01_4MM2_BLUE
- removed J184: 47, symbol Beatrice:Conn_02x01_24VDC
- removed J185: 45, symbol Beatrice:Conn_02x01_4MM2_GREY
- removed J193: 48, symbol Beatrice:Conn_02x01_24VDC
- removed J2: 42, symbol Beatrice:Conn_02x01_24VDC
- removed J215: 30, symbol Beatrice:Conn_02x01_4MM2_GREY
- removed J222: 50, symbol Beatrice:Conn_02x01_24VDC
- removed J242: 63, symbol Beatrice:Conn_02x01_4MM2_GREY
- removed J247: 60, symbol Beatrice:Conn_02x01_4MM2_GREY
- removed J291: 07, symbol Beatrice:Conn_02x01_4MM2_GREY
- removed J293: 08, symbol Beatrice:Conn_02x01_4MM2_GREY
- removed J309, J310: 20, symbol Beatrice:Conn_02x01_24VDC
- removed J313: 08, symbol Beatrice:Conn_02x01_4MM2_BLUE
- removed RL10: ANCHOR LIGHT RELAY (AL), symbol Relay:FINDER-40.52
- removed RL4: COURTESY LIGHTS RELAY (CTL), symbol Relay:FINDER-40.52
- removed RL7: NMEA BUS 1 RELAY (N1), symbol Relay:FINDER-40.52
- removed RL8: WORK LIGHT RELAY (WL), symbol Relay:FINDER-40.52
- removed U2: PANEL DIMMER (HPD), symbol Beatrice:PanelDimmer
- added J11: 04, symbol Beatrice:Conn_02x01_4MM2_BLUE
- added J12, J19: 05, symbol Beatrice:Conn_02x01_4MM2_BLUE
- added J13, J44: 06, symbol Beatrice:Conn_02x01_4MM2_BLUE
- added J14, J20, J45: 07, symbol Beatrice:Conn_02x01_4MM2_BLUE
- added J15: 03, symbol Beatrice:Conn_02x01_4MM2_GREY
- added J16, J46: 08, symbol Beatrice:Conn_02x01_4MM2_BLUE
- added J17, J30: 10, symbol Beatrice:Conn_02x01_4MM2_BLUE
- added J18: 09, symbol Beatrice:Conn_02x01_4MM2_BLUE
- added J2: 48, symbol Beatrice:Conn_02x01_4MM2_GREY
- added J21, J40: 01, symbol Beatrice:Conn_02x01_4MM2_BLUE
- added J22: 11, symbol Beatrice:Conn_02x01_4MM2_BLUE
- added J23: 12, symbol Beatrice:Conn_02x01_4MM2_BLUE
- added J24: 13, symbol Beatrice:Conn_02x01_4MM2_BLUE
- added J25: 14, symbol Beatrice:Conn_02x01_4MM2_BLUE
- added J26: 15, symbol Beatrice:Conn_02x01_4MM2_BLUE
- added J27, J34: 13, symbol Beatrice:Conn_03x01
- added J28: 12, symbol Beatrice:Conn_02x01_24VDC
- added J29: 13, symbol Beatrice:Conn_02x01_24VDC
- added J35: 33, symbol Beatrice:Conn_02x01_24VDC
- added J36: 50, symbol Beatrice:Conn_02x01_4MM2_GREY
- added J37: 29, symbol Beatrice:Conn_02x01_4MM2_GREY
- added J38: 47, symbol Beatrice:Conn_02x01_4MM2_GREY
- added J39: 02, symbol Beatrice:Conn_02x01_4MM2_BLUE
- added K4, K5, K6, K7, K8, K9: FINDER-32.21-x000, Relay_THT:Relay_SPDT_Finder_32.21-x000, symbol Relay:FINDER-32.21-x000
- added U6: PANEL DIMMER (HPD), symbol Beatrice:PanelDimmer
- J1: value 20 -> 19
- J10: value 06 -> 07
- J147: value 05 -> 09
- J151: value 05 -> 03
- J152: value 06 -> 04
- J155: value 10 -> 11
- J158: value 16 -> 14
- J159: value 20 -> 18
- J160: value 21 -> 20
- J161: value 08 -> 12
- J162: value 25 -> 24
- J164: value 39 -> 40
- J165: value 13 -> 11
- J166: value 32 -> 30
- J167: value 11 -> 14
- J170: value 41 -> 37
- J171: value 43 -> 35
- J172: value 44 -> 36
- J174: value 51 -> 22
- J175: value 18 -> 16
- J176: value 19 -> 17
- J178: value 53 -> 24
- J179: value 10 -> 13
- J181: value 55 -> 42
- J182: value 56 -> 43
- J183: value 46 -> 41
- J188: value 12 -> 10
- J189: value 36 -> 34
- J190: value 37 -> 39
- J191: value 62 -> 32
- J192: value 13 -> 02
- J194: value 07 -> 11
- J195: value 14 -> 03
- J196: value 42 -> 38
- J197: value 31 -> 29
- J198: value 33 -> 31
- J200: value 02 -> 04
- J201: value 03 -> 15
- J202: value 04 -> 05
- J203: value 05 -> 06
- J204: value 34 -> 32
- J205: value 06 -> 08
- J206: value 35 -> 33
- J207: value 07 -> 09
- J208: value 24 -> 23
- J209: value 52 -> 23
- J210: value 28 -> 27
- J211: value 11 -> 09
- J212: value 23 -> 22
- J213: value 10 -> 08
- J214: value 29 -> 28
- J216: value 26 -> 25
- J217: value 27 -> 26
- J218: value 17 -> 15
- J219: value 22 -> 21
- J220: value 14 -> 16
- J221: value 21 -> 02
- J223: value 15 -> 17
- J224: value 16 -> 18
- J225: value 17 -> 06
- J226: value 23 -> 28
- J228: value 11 -> 12
- J232: value 12 -> 13
- J234: value 17 -> 19
- J235: value 18 -> 20
- J236: value 19 -> 21
- J237: value 13 -> 14
- J238: value 22 -> 27
- J239: value 65 -> 51
- J241: value 12 -> 01
- J243: value 61 -> 31
- J244: value 57 -> 44
- J245: value 58 -> 45
- J246: value 59 -> 46
- J248: value 18 -> 07
- J249: value 19 -> 08
- J250: value 24 -> 30
- J251: value 25 -> 34
- J270: value 06 -> 10
- J294: value 03 -> 01
- J295: value 04 -> 02
- J3: value 53 -> 25
- J307: value 64 -> 49
- J4: value 53 -> 26
- J6: value 15 -> 04
- J60: value 01 -> 03
- J7: value 16 -> 05
- J8: value 06 -> 05
- RL1: value SPUD ISOLATOR RELAY (SPD) -> NMEA BUS 0 RELAY (N0R)
- RL3: value VHF RELAY (VH) -> VHF RELAY (VHR)
- RL6: value NMEA BUS 0 RELAY (N0) -> NMEA BUS 0 RELAY (N0R)
Connections:
- net AIS.+24VDC is gone; now on net HP.F9.1.3.AIS.OP1: J60. (Pin_2)
- net BLUEBOARD_+/- is gone; now on net HP.F9.2.3.A: J202. (Pin_2)
- net BLUEBOARD_-/+ is gone; now on net HP.F9.2.3.B: J203. (Pin_2)
- net DP.GND.CTL.OP1 is gone; now on net GND.CTL: J188. (Pin_2)
- net F9.1.4.SB is gone; now on net F9.1.4.CTL.A: J205. (Pin_2)
- net F9.1.5.AL.A is gone; now on net F9.1.5.ANL.A: J201. (Pin_2)
- net F9.1.5.AL.B is gone; now on net NMEA_INTERFACE1_+: U3. (CANBUS)
- net F9.1.6.NO (24VDC VHF SUPPLY) is gone; now on net F9.1.6.NO: RL3.14
- net F9.1.8.SPD.A is gone; now on net F9.3.5: RL1.11
- net F9.1.8.SPD.B is gone; now on net F9.3.6: RL1.21
- net F9.1.8.SPUD.B is gone; now on net SPUD_ISOLATOR_+/-: J221. (Pin_2)
- net F9.3.7.NO (12VDC VHF SUPPLY) is gone; now on net F9.3.7.NO: RL3.24
- net HP.GND.HPD.PWM is gone; now on net HPD.SBY.PWM: J287. (Pin_2)
- net HP.GND.HPD.PWM.INT is gone; now on net HPD.SBY.PWM.INT: J288. (Pin_2)
- net HP.IN02.T09 is gone; now on net GND.NB0: J190. (Pin_2), RL6.A1
- net HP.IN02.T11 is gone; now on net GND.NB1: J164. (Pin_2)
- net NMEA_ETH.IO5G is gone; now on net WL.COIL.RM: U5. (R4-NO)
- net RADAR_ON is gone; now on net RADAR_+: J235. (Pin_2)
- net WIFI_ON is gone; now on net WIFI_+: J250. (Pin_2)
- net WIPER_MODE is gone; now on net WIPER_ON (BROWN): J191. (Pin_2)
- net WIPER_ON is gone; now on net WIPER_CTL (BLACK): J243. (Pin_2)
- net WL.COIL is gone; now on net HP.GND.WNL: J307. (Pin_2)
- net WORK_LIGHT_+ is gone; now on net WORK LIGHT (1): J251. (Pin_2)
- net F9.1.2: no longer RL6.A2
- net F9.1.4: now also K7.11, K7.A2, K9.11, K9.A2
- net F9.1.5: now also K4.11, K4.A2
- net F9.1.8: now also J19. (Pin_2); no longer RL1.14, RL1.22, RL1.A1
- net F9.1.9: now also K5.11, K5.A2
- net F9.2.6: now also K6.11, K6.A2
- net F9.3.3: no longer J220. (Pin_2), J6. (Pin_2)
- net F9.3.4: no longer J223. (Pin_2)
- net F9.3.5: no longer J224. (Pin_2), J7. (Pin_2)
- net F9.3.6: no longer J234. (Pin_2)
- net GND: now also J5. (Pin_2), K2.A1, U6. (SUPPLY); no longer RL1.12, RL1.24
- net HP.F9.1.7.WIF.OP1: now also J250. (Pin_2)
- net HP.F9.2.5.RDR.OP1: now also J235. (Pin_2)
- net HP.F9.2.8.THR.ACT: now also J209. (Pin_2); no longer J178. (Pin_2)
- net HP.F9.2.8.THR.RGT: now also J178. (Pin_2); no longer J209. (Pin_2)
- net HP.GND.RPM.ALM: now also J23. (Pin_2)
- net HP.IGN.75.TRL.SBY: now also J22. (Pin_2)
- net HP.IGN.75.TRL.SBY.A: now also J25. (Pin_2)
- net HP.IGN.75.TRL.SBY.B: now also J24. (Pin_2)
- net HPD.DEC: now also U6. (SUPPLY)
- net HPD.INC: now also U6. (SUPPLY)
- net IGN.75.TRL.SBY: now also J22. (Pin_2); no longer K3.11, K3.A2
- net IGN.75.TRL.SBY.A: now also U4. (CANBUS), J25. (Pin_2), J26. (Pin_2)
- net IGN.75.TRL.SBY.B: now also J24. (Pin_2); no longer U4. (CANBUS)
- net NMEA_0.01: now also J206. (Pin_2); no longer J204. (Pin_2)
- net NMEA_0.02: now also J211. (Pin_2); no longer J206. (Pin_2)
- net NMEA_0.03: now also J213. (Pin_2); no longer J211. (Pin_2)
- net NMEA_0.04: now also J197. (Pin_2); no longer J213. (Pin_2)
- net NMEA_0.05: now also J166. (Pin_2); no longer J197. (Pin_2)
- net NMEA_0.06: now also J198. (Pin_2); no longer J166. (Pin_2)
- net NMEA_0.07: now also J27. (Pin_2); no longer J198. (Pin_2)
- net NMEA_0.08: now also J34. (Pin_2)
- net NMEA_0.11: now also J176. (Pin_2); no longer J175. (Pin_2)
- net NMEA_0.12: now also J158. (Pin_2); no longer J176. (Pin_2)
- net NMEA_0.13: no longer J158. (Pin_2)
- net NMEA_0.14: now also J216. (Pin_2)
- net NMEA_0.15: now also J212. (Pin_2); no longer J216. (Pin_2)
- net NMEA_1.02: now also J182. (Pin_2); no longer J181. (Pin_2)
- net NMEA_1.03: now also J244. (Pin_2); no longer J182. (Pin_2)
- net NMEA_1.04: now also J245. (Pin_2); no longer J244. (Pin_2)
- net NMEA_1.05: now also J294. (Pin_2); no longer J245. (Pin_2)
- net NMEA_1.06: now also J295. (Pin_2); no longer J294. (Pin_2)
- net NMEA_1.07: now also J171. (Pin_2); no longer J295. (Pin_2)
- net NMEA_1.08: now also J172. (Pin_2); no longer J171. (Pin_2)
- net NMEA_1.09: now also J4. (Pin_2); no longer J172. (Pin_2)
- net NMEA_1.10: now also J16. (Pin_2), J18. (Pin_2); no longer J3. (Pin_2)
- net NMEA_1.13: now also J208. (Pin_2)
- net NMEA_ETH.IO5P: no longer U5. (R4-NO)
- net SOLENOID R: now also J178. (Pin_2); no longer J209. (Pin_2)
- net SPUD_ISOLATOR_+/-: now also J21. (Pin_2)
- net at D1.1 (K), D2.1 (K): now also J209. (Pin_2); no longer J178. (Pin_2)
- net AIS.RECEIVE_ONLY renamed HP.F9.1.3.AIS.OP2
- removed net AL.COIL.RM: J151. (Pin_2), J152. (Pin_2), U5. (R4-NO)
- net ANCHOR_LIGHT(WHEELHOUSE)_+ renamed F9.1.5.ANL.A
- net F9.1.5.ANL.A: now also U5. (R4-NO), J34. (Pin_2)
- net BLUE-BOARD-BLACK renamed HP.F9.2.3.B
- net HP.F9.2.3.B: no longer U4. (CANBUS)
- net BLUE-BOARD-RED renamed HP.F9.2.3.A
- net CTL.COIL.RM renamed GND.CTL
- net GND.CTL: now also K9.A1
- removed net F5.1.7.HPD.SBY: J5. (Pin_2), K2.A1
- net F9.1.1.DP.SW(ANCHOR_LIGHT).P1NO renamed GND.ANL
- net GND.ANL: now also J152. (Pin_2), U5. (R4-NO), K4.A1
- net F9.1.1.DP.SW(HELM).P1NO renamed HP.GND.HIS
- net F9.1.1.DP.SW(NAVIGATION LIGHTS).P1NO renamed GND.NVL
- net GND.NVL: now also J196. (Pin_2), RL2.A1
- net F9.1.1.DP.SW(NMEA_BUS_0).P1NO renamed GND.NB0
- net F9.1.1.DP.SW(NMEA_BUS_1).P1NO renamed GND.NB1
- net GND.NB1: now also RL1.A1
- net F9.1.1.DP.SW(VHF).P1NO renamed HP.GND.VHF
- net F9.1.4 (COURTESY LIGHTS) renamed F9.1.4 (COURTESY/NIGHT LIGHTS)
- net F9.1.4.PS renamed F9.1.4.CTL.A
- net F9.1.4.CTL.A: now also K9.14
- removed net F9.1.5.NL.A: J228. (Pin_2), J232. (Pin_2), J237. (Pin_2), RL2.14
- net F9.1.5.NL.B renamed NMEA_0.09
- net F9.1.9.WL renamed WORK LIGHT (1)
- net F9.2.4 (SPARE) renamed F9.2.4 (DECK LIGHTS)
- net F9.3.1 (NMEA INTERFACES) renamed F9.3.1 (NMEA MODULE SUPPLY)
- net F9.3.3 (NMEA BUS 0 LEG A SUPPLY) renamed F9.3.3.NB0
- net F9.3.3.NB0: now also J220. (Pin_2)
- net F9.3.4 (NMEA BUS 0 LEG B SUPPLY) renamed F9.3.4.NB0
- net F9.3.4.NB0: now also J223. (Pin_2)
- net GND.HPD.PWM renamed HPD.SBY.PWM
- net HPD.SBY.PWM: now also U6. (SUPPLY)
- net GND.HPD.PWM.INT renamed HPD.SBY.PWM.INT
- net GROUND.DP.MIRSW.P1NO renamed HP.GND.MIS
- net HI.COIL renamed GND.HIS
- net HORN-ON renamed HP.F9.1.11.OP1 (HORN)
- net HP.F9.2.6.SRL.OP1 renamed HP.GND.SRL
- net HP.F9.2.7.WPR.CFG renamed WIPER_ON (BROWN)
- net HP.F9.2.7.WPR.OP1 renamed WIPER_CTL (BLACK)
- net HP.GND.ANL.OP1 renamed HP.GND.ANL
- net HP.GND.CTL.OP1 renamed HP.GND.CTL
- net HP.GND.NVL.OP1 renamed HP.GND.NVL
- net HP.GND.WKL.OP1 renamed HP.GND.WNL
- net HP.VHF_+ renamed IC-M577-POS
- net MI.COIL renamed GND.MIS
- removed net NL.COIL.RM: J170. (Pin_2), J196. (Pin_2), RL2.A1, U5. (R4-NO)
- removed net NMEA_0.16: J212. (Pin_2), U3. (CANBUS)
- removed net NMEA_1.14: J208. (Pin_2), U4. (CANBUS)
- net SEARCHLIGHT_+ renamed SEARCH LIGHT (2)
- removed net SEARCHLIGHT_ON: J183. (Pin_2), J236. (Pin_2)
- net SPD.COIL.SW renamed F9.3.1.R
- net F9.3.1.R: now also RL6.A2
- net STEAMING_LIGHT(WHEELHOUSE)_+ renamed STEAMING LIGHT (3)
- net TSR.COIL renamed GND.RPM.ALM
- net GND.RPM.ALM: now also J23. (Pin_2)
- net VH.COIL renamed GND.VHF
- new net: J27. (Pin_2), K8.14
- new net: J34. (Pin_2), K4.14
- new net: J261. (Pin_2), J262. (Pin_2)
- new net: J266. (Pin_2), J269. (Pin_2)
- new net (n/c): J239. (Pin_2), J30. (Pin_2), J37. (Pin_2)
- new net ANCHOR LIGHT (4): J201. (Pin_2)
- new net B.BOARD-NEG/POS: J20. (Pin_2), J203. (Pin_2), U4. (CANBUS)
- new net B.BOARD-POS/NEG: J202. (Pin_2)
- new net DP.GND.ANL: J151. (Pin_2)
- new net DP.GND.CTL: J188. (Pin_2)
- new net DP.GND.DKL: J28. (Pin_2)
- new net DP.GND.NB0: J190. (Pin_2)
- new net DP.GND.NB1: J164. (Pin_2)
- new net DP.GND.NVL: J170. (Pin_2)
- new net F9.1.10: J44. (Pin_2), J45. (Pin_2), J46. (Pin_2)
- new net F9.1.4.WNL.A: J37. (Pin_2), K7.14
- new net F9.1.5.ANL: U5. (R4-NO)
- new net F9.1.5.NVL.A: J228. (Pin_2), J232. (Pin_2), RL2.14
- new net F9.1.5.NVL.B: U5. (R4-NO)
- new net F9.1.5.STL: J237. (Pin_2), U5. (R4-NO)
- new net F9.1.9.WKL.A: J251. (Pin_2), K5.14
- new net F9.2.4: K8.11, K8.A2
- new net F9.2.4.DKL.A: J27. (Pin_2), J30. (Pin_2)
- new net F9.2.6.SRL.A: J236. (Pin_2), K6.14
- new net F9.3.3.N0R.HP: J6. (Pin_2)
- new net F9.3.5.N1R.HP: J7. (Pin_2)
- new net F9.3.5.NB1: J224. (Pin_2), RL1.14
- new net F9.3.6.NB1: J234. (Pin_2), RL1.24
- new net GND.DKL: J28. (Pin_2), J29. (Pin_2), K8.A1
- new net GND.SRL: J183. (Pin_2), K6.A1
- new net GND.WKL: J2. (Pin_2), J38. (Pin_2), K5.A1
- new net GND.WNL: J307. (Pin_2), J36. (Pin_2), K7.A1
- new net HP.F9.1.8: J19. (Pin_2)
- new net HP.F9.1.8.A: J21. (Pin_2)
- new net HP.F9.1.8.B: J221. (Pin_2)
- new net HP.F9.2.7.CO (WIPER): J243. (Pin_2)
- new net HP.F9.2.7.OP1 (WIPER): J191. (Pin_2)
- new net HP.F9.2.7.OP2 (WIPER): J35. (Pin_2)
- new net HP.GND.DKL: J29. (Pin_2)
- new net HP.GND.WKL: J38. (Pin_2)
- new net HP.HPD.SBY.PWM: J287. (Pin_2)
- new net HP.HPD.SBY.PWM.INT: J288. (Pin_2)
- new net HP.SP.ALM.LED (6): J17. (Pin_2)
- new net HP.SP.DN (3): J13. (Pin_2)
- new net HP.SP.DN.LED (5): J16. (Pin_2)
- new net HP.SP.GND (G/Y): J15. (Pin_2)
- new net HP.SP.POS (1): J11. (Pin_2)
- new net HP.SP.UP (2): J12. (Pin_2)
- new net HP.SP.UP.LED (4): J14. (Pin_2)
- new net Little green wire???: J45. (Pin_2)
- new net NMEA_0.00: J204. (Pin_2), U3. (CANBUS)
- new net NMEA_0.10: J175. (Pin_2), U3. (CANBUS)
- new net NMEA_1.01: J181. (Pin_2), U4. (CANBUS)
- new net REM.GND.NVL: U5. (R4-NO)
- new net SP.ALM.LED (6): J17. (Pin_2)
- new net SP.DN (3): J13. (Pin_2)
- new net SP.GND (G/Y): J15. (Pin_2)
- new net SP.POS (1): J11. (Pin_2)
- new net SP.UP (2): J12. (Pin_2)
- new net SP.UP.LED (4): J14. (Pin_2)
- new net TSR.IGN.75.TRL.SBY: K3.11, K3.A2
- new net WIPER_MODE (GREY): J35. (Pin_2)
- no-connect marks 3 -> 1
Other:
- note removed: "12 VDC SIGNAL"
- note removed: "12VDC"
- note removed: "24VDC"
- note removed: "24VDC PWM"
- note removed: "24VDC SIGNAL"
- note removed: "GND"
- note removed: "GND PWM"
- note removed: "The Courtesy Light Relay (CLR) switches power to the wheelhouse courtesy lights and is operated by physical switches at the helm and domestic panels and by an NMEA modulated remote relay."
