File: resources/kicad/schematics/dc/helm/troll-system.kicad_sch (KiCad schematic)
At the start: 27 parts, among them J1 Conn_01x02_Pin, J10 Conn_01x02_Socket, J11 Conn_01x02_Socket, J12 Conn_01x02_Socket, J13 Conn_01x02_Pin, J14 Conn_01x02_Pin, J15 Conn_01x02_Pin, J16 Conn_01x02_Pin, J17 Conn_01x03_Socket, J18 Conn_01x03_Pin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

Commit message: Refactor
Connections:
- net at J10.1 (Pin_1), J18.3 (Pin_3), U2.16 (GND)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: now also J9.2 (Pin_2)
- net at U2.10 (SDA/AN): now also J18.1 (Pin_1)
- net at U2.13 (RX): no longer J9.1 (Pin_1)
- net at U2.14 (RC): no longer J18.1 (Pin_1)
- net at U2.15 (5V): no longer J9.2 (Pin_2)
- net at U2.9 (SCL): now also J9.1 (Pin_1)
Other:
- note added: "17"
- note removed: "14"
- moved on the sheet: D1
Changed lines of the file:
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@@
+	)
+	(junction
+		(at 162.56 72.39)
+		(diameter 0)
+		(color 0 0 0 0)
 	)
 	(junction
@@
 	(wire
 		(pts
+			(xy 149.86 54.61) (xy 171.45 54.61)
+		)
+		(stroke
+			(width 0)
+			(type default)
+		)
+	)
+	(wire
+		(pts
 			(xy 226.06 80.01) (xy 234.95 80.01)
 		)
@@
 	(wire
 		(pts
-			(xy 149.86 44.45) (xy 149.86 72.39)
-		)
-		(stroke
-			(width 0)
-			(type default)
-		)
-	)
-	(wire
-		(pts
 			(xy 247.65 46.99) (xy 245.11 46.99)
 		)
@@
 	(wire
 		(pts
+			(xy 162.56 72.39) (xy 162.56 77.47)
+		)
+		(stroke
+			(width 0)
+			(type default)
+		)
+	)
+	(wire
+		(pts
 			(xy 119.38 78.74) (xy 119.38 77.47)
 		)
@@
 	(wire
 		(pts
-			(xy 104.14 52.07) (xy 104.14 60.96)
-		)
-		(stroke
-			(width 0)
-			(type default)
-		)
-	)
-	(wire
-		(pts
-			(xy 149.86 44.45) (xy 171.45 44.45)
+			(xy 104.14 52.07) (xy 104.14 58.42)
 		)
 		(stroke
@@
 	(wire
 		(pts
-			(xy 165.1 72.39) (xy 215.9 72.39)
-		)
-		(stroke
-			(width 0)
-			(type default)
-		)
-	)
-	(wire
-		(pts
 			(xy 245.11 72.39) (xy 251.46 72.39)
 		)
@@
 	(wire
 		(pts
-			(xy 104.14 68.58) (xy 104.14 71.12)
+			(xy 104.14 66.04) (xy 104.14 71.12)
 		)
 		(stroke
@@
 	(wire
 		(pts
-			(xy 171.45 41.91) (xy 165.1 41.91)
-		)
-		(stroke
-			(width 0)
-			(type default)
-		)
-	)
-	(wire
-		(pts
 			(xy 245.11 77.47) (xy 255.27 77.47)
 		)
@@
 	(wire
 		(pts
-			(xy 167.64 69.85) (xy 167.64 46.99)
-		)
-		(stroke
-			(width 0)
-			(type default)
-		)
-	)
-	(wire
-		(pts
-			(xy 167.64 46.99) (xy 171.45 46.99)
+			(xy 167.64 69.85) (xy 167.64 57.15)
 		)
 		(stroke
@@
 	(wire
 		(pts
+			(xy 149.86 54.61) (xy 149.86 72.39)
+		)
+		(stroke
+			(width 0)
+			(type default)
+		)
+	)
+	(wire
+		(pts
 			(xy 149.86 74.93) (xy 152.4 74.93)
 		)
@@
 	(wire
 		(pts
-			(xy 162.56 39.37) (xy 162.56 77.47)
+			(xy 162.56 39.37) (xy 162.56 72.39)
 		)
 		(stroke
@@
 	(wire
 		(pts
+			(xy 162.56 72.39) (xy 215.9 72.39)
+		)
+		(stroke
+			(width 0)
+			(type default)
+		)
+	)
+	(wire
+		(pts
 			(xy 205.74 77.47) (xy 205.74 59.69)
 		)
@@
 	(wire
 		(pts
-			(xy 165.1 41.91) (xy 165.1 72.39)
+			(xy 167.64 57.15) (xy 171.45 57.15)
 		)
 		(stroke
@@
 		)
 	)
-	(text_box "The system is powered directly from the main engine\nignition switch via the Troll System Relay (TSR) mounted\nin the helm cabinet. TSR provides two power rails:\n\nHP.ENG.IGN.SBY is live when the engine ignition switch\nis ON and engine RPMs are below the tachometer alarm\nthreshold. This supply is used to power the troll\nsystem.\n\nHP.ENG.IGN.ALM is live when the engine ignition switch\nis ON and engine RPMs are above the tachometer alarm\nthreshold. This supply is used to power the troll\nsystem overspeed alarm LED.\n"
+	(text_box "The troll valve system is powered from the main engine\nignition switch auxilliary supply ENG.IGN via the Troll\nSystem Relay (TSR) mounted in the helm cabinet. TSR\nprovides two power rails:\n\nHP.ENG.IGN.SBY is live when the engine ignition switch\nis ON and engine RPMs are below the tachometer alarm\nthreshold. This supply is used to power the troll\nsystem.\n\nHP.ENG.IGN.ALM is live when the engine ignition switch\nis ON and engine RPMs are above the tachometer alarm\nthreshold. This supply is used to power the troll\nsystem overspeed alarm LED.\n"
 		(exclude_from_sim no)
 		(at 14.605 90.17 0)
@@
 		)
 	)
-	(text "14"
+	(text "17"
 		(exclude_from_sim no)
 		(at 128.27 72.39 0)
@@
 	(symbol
 		(lib_id "Device:LED")
-		(at 104.14 64.77 270)
+		(at 104.14 62.23 270)
 		(unit 1)
 		(exclude_from_sim no)
@@
 		(dnp no)
 		(property "Reference" "D1"
-			(at 101.1682 64.5922 90)
+			(at 101.1682 62.0522 90)
 			(effects
 				(font
@@
 		)
 		(property "Value" "LED"
-			(at 101.1682 63.4492 90)
+			(at 101.1682 60.9092 90)
 			(effects
 				(font
@@
 		)
 		(property "Footprint" ""
-			(at 104.14 64.77 0)
+			(at 104.14 62.23 0)
 			(effects
 				(font
@@
 		)
 		(property "Datasheet" "~"
-			(at 104.14 64.77 0)
+			(at 104.14 62.23 0)
 			(effects
 				(font
@@
 		)
 		(property "Description" ""
-			(at 104.14 64.77 0)
-			(effects
-				(font
+			(at 104.14 62.23 0)
+			(effects
+				(font

Commit message: Updates
Parts:
- added R1: R_Small, symbol Device:R_Small
- D1: value LED -> ALARM
Connections:
- net HP.ENG.IGN.ALM: now also R1.2; no longer D1.2 (A)
- new net: D1.2 (A), R1.1
Other:
- moved on the sheet: D1
Changed lines of the file:
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@@
 		(date "2020-01-06")
 		(rev "1")
+		(comment 1 "See helm schematic for details of power supply switching.")
 	)
 	(junction
@@
 	(wire
 		(pts
-			(xy 104.14 52.07) (xy 104.14 58.42)
+			(xy 104.14 52.07) (xy 104.14 54.61)
 		)
 		(stroke
@@
 	(wire
 		(pts
-			(xy 104.14 66.04) (xy 104.14 71.12)
-		)
-		(stroke
-			(width 0)
-			(type default)
-		)
-	)
-	(wire
-		(pts
 			(xy 247.65 54.61) (xy 247.65 46.99)
 		)
@@
 	(wire
 		(pts
+			(xy 104.14 67.31) (xy 104.14 71.12)
+		)
+		(stroke
+			(width 0)
+			(type default)
+		)
+	)
+	(wire
+		(pts
 			(xy 90.17 59.69) (xy 90.17 74.93)
 		)
@@
 		)
 	)
-	(text_box "System Supply"
+	(text_box "Helm"
 		(exclude_from_sim no)
 		(at 14.605 21.59 0)
@@
 		)
 	)
-	(text_box "HELM PANEL"
+	(text_box "WHEELHOUSE"
 		(exclude_from_sim no)
 		(at 14.605 15.24 0)
@@
 		)
 	)
-	(text_box "A POLOLU stepper controller drives a stepper motor in step with the joystick position. The\nstepper motor spindle is coupled to the hydraulic valve spindle. A microswitch detects\nspindle position and allows the controller to properly initialise the stepper motor.\n\n "
+	(text_box "A POLOLU stepper controller drives a stepper motor in step with the joystick\nposition. \n "
 		(exclude_from_sim no)
 		(at 143.51 90.17 0)
@@
 		)
 	)
-	(text_box "The trolling system implements an electronic control interface to a hydraulic trolling valve.\n\nThe engine control panel ignition-on terminal provides all system power.  "
-		(exclude_from_sim no)
-		(at 14.605 127 0)
-		(size 158.75 64.77)
-		(stroke
-			(width 0)
-			(type default)
-		)
-		(fill
-			(type none)
-		)
-		(effects
-			(font
-				(size 1.27 1.27)
-			)
-			(justify left top)
-		)
-	)
-	(text_box "The troll valve system is powered from the main engine\nignition switch auxilliary supply ENG.IGN via the Troll\nSystem Relay (TSR) mounted in the helm cabinet. TSR\nprovides two power rails:\n\nHP.ENG.IGN.SBY is live when the engine ignition switch\nis ON and engine RPMs are below the tachometer alarm\nthreshold. This supply is used to power the troll\nsystem.\n\nHP.ENG.IGN.ALM is live when the engine ignition switch\nis ON and engine RPMs are above the tachometer alarm\nthreshold. This supply is used to power the troll\nsystem overspeed alarm LED.\n"
+	(text_box "The troll valve system receives power from two 24VDC\nsupply rails which are enabled only when the engine\nignition switch is in the ACC position and the helm\nTROLL switch is ON.\n\nHP.ENG.IGN.SBY is the normal system supply and is live\nwhen engine RPMs are BELOW the tachometer alarm\nthreshold.\n\nHP.ENG.IGN.ALM is an alarm signal which is asserted\nonly when engine RPM is ABOVE the tachometer alarm\nthreshold. This supply is used to power an LED indicator\nwhich alerts the user when the troll system is\nunavailable because of RPM overspeed.\n\n"
 		(exclude_from_sim no)
 		(at 14.605 90.17 0)
@@
 		)
 	)
+	(text_box "The stepper motor spindle is coupled directly to\nthe trolling valve operating spindle. A cam operated\nmicroswitch detects spindle position and provides\nlimit feedback to the Pololu controller.\n\nThe trolling valve isolation valve is opened\nimmedaitely power is applied to the troll system.\n"
+		(exclude_from_sim no)
+		(at 231.14 90.17 0)
+		(size 51.435 31.75)
+		(stroke
+			(width -0.0001)
+			(type default)
+		)
+		(fill
+			(type none)
+		)
+		(effects
+			(font
+				(size 1.27 1.27)
+			)
+			(justify left top)
+		)
+	)
 	(text_box "Troll Valve Actuator"
 		(exclude_from_sim no)
@@
 		)
 	)
-	(text_box "When the system is powered, a voltage regulator\nproduces a 5V output which feeds the positive\nrail of a joystick operated potentiometer. Wiper\noutput from the potentiometer is fed via the\nengine loom to the engine connection cabinet."
+	(text_box "The helm troll panel includes a 78L05 voltage\nregulator which produces a 5V output feeding the\npositive rail of a joystick operated potentiometer.\n\nWiper output from the potentiometer is fed via the\nengine loom to the engine connection cabinet."
 		(exclude_from_sim no)
 		(at 74.295 90.17 0)
@@
 	(symbol
 		(lib_id "Device:LED")
-		(at 104.14 62.23 270)
+		(at 104.14 58.42 270)
 		(unit 1)
 		(exclude_from_sim no)
@@
 		(dnp no)
 		(property "Reference" "D1"
-			(at 101.1682 62.0522 90)
-			(effects
-				(font
-					(size 1.27 1.27)
-				)
-				(justify right)
-			)
-		)
-		(property "Value" "LED"
-			(at 101.1682 60.9092 90)
-			(effects
-				(font
-					(size 1.27 1.27)
-				)
-				(justify right)
-				(hide yes)
+			(at 100.838 57.912 90)
+			(effects
+				(font
+					(size 1.27 1.27)
+				)
+			)
+		)
+		(property "Value" "ALARM"
+			(at 109.22 57.912 90)
+			(effects
+				(font
+					(size 1.27 1.27)
+				)
 			)
 		)
 		(property "Footprint" ""
-			(at 104.14 62.23 0)
+			(at 104.14 58.42 0)
 			(effects
 				(font
@@
 		)
 		(property "Datasheet" "~"
-			(at 104.14 62.23 0)
+			(at 104.14 58.42 0)
 			(effects
 				(font
@@
 		)
 		(property "Description" ""
-			(at 104.14 62.23 0)
+			(at 104.14 58.42 0)
 			(effects
 				(font
@@
 					(unit 1)
 				)
+			)
+		)
+	)
+	(symbol
+		(lib_id "Device:R_Small")
+		(at 104.14 64.77 0)
+		(unit 1)
+		(exclude_from_sim no)
+		(in_bom yes)
+		(on_board yes)
+		(dnp no)
+		(property "Reference" "R1"
+			(at 100.838 64.516 0)
+			(effects
+				(font
+					(size 1.27 1.27)
+				)
+			)
+		)
+		(property "Value" "R_Small"
+			(at 106.68 66.0399 0)
+			(effects
+				(font
+					(size 1.27 1.27)
+				)
+				(justify left)
+				(hide yes)
+			)
+		)
+		(property "Footprint" ""
+			(at 104.14 64.77 0)
+			(effects
+				(font
+					(size 1.27 1.27)
+				)
+				(hide yes)
+			)
+		)
+		(property "Datasheet" "~"
+			(at 104.14 64.77 0)
+			(effects
+				(font
+					(size 1.27 1.27)
+				)
+				(hide yes)
+			)
+		)
+		(property "Description" "Resistor, small symbol"
+			(at 104.14 64.77 0)
+			(effects
+				(font
+					(size 1.27 1.27)
+				)
+				(hide yes)
+			)
+		)
+		(pin "1"
+		)
+		(pin "2"
+		)
+		(instances
+			(project ""
+				(path "/80df189f-0b25-47f8-986e-6f92283f20c3"
+					(reference "R1")
+					(unit 1)
+				)

Commit message: Many tweaks
Connections:
- net HP.ENG.IGN.SBY is gone; now on net HP.IGN.75.TRL.SBY.B: J17.2 (Pin_2), U1.8 (IN)
- net GND: no longer D1.1 (K), RV1.1
- net HP.ENG.IGN.ALM renamed HP.IGN.75.TRL.SBY.B
- new net HP.IGN.75.TRL.SBY.A: D1.1 (K)
Other:
- moved on the sheet: D1, R1
Changed lines of the file:
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@@
-	)
-	(junction
-		(at 104.14 52.07)
-		(diameter 0)
-		(color 0 0 0 0)
 	)
 	(junction
@@
 	)
 	(junction
+		(at 111.76 74.93)
+		(diameter 0)
+		(color 0 0 0 0)
+	)
+	(junction
 		(at 205.74 77.47)
 		(diameter 0)
@@
 	(wire
 		(pts
+			(xy 111.76 55.88) (xy 111.76 58.42)
+		)
+		(stroke
+			(width 0)
+			(type default)
+		)
+	)
+	(wire
+		(pts
 			(xy 226.06 80.01) (xy 234.95 80.01)
 		)
@@
 	(wire
 		(pts
+			(xy 111.76 71.12) (xy 111.76 74.93)
+		)
+		(stroke
+			(width 0)
+			(type default)
+		)
+	)
+	(wire
+		(pts
 			(xy 260.35 74.93) (xy 260.35 73.66)
 		)
@@
 	(wire
 		(pts
-			(xy 104.14 52.07) (xy 104.14 54.61)
-		)
-		(stroke
-			(width 0)
-			(type default)
-		)
-	)
-	(wire
-		(pts
 			(xy 252.73 44.45) (xy 245.11 44.45)
 		)
@@
 	(wire
 		(pts
-			(xy 97.79 52.07) (xy 104.14 52.07)
+			(xy 97.79 52.07) (xy 119.38 52.07)
 		)
 		(stroke
@@
 	(wire
 		(pts
-			(xy 121.92 72.39) (xy 132.08 72.39)
+			(xy 124.46 72.39) (xy 132.08 72.39)
 		)
 		(stroke
@@
 	(wire
 		(pts
-			(xy 90.17 74.93) (xy 132.08 74.93)
+			(xy 90.17 74.93) (xy 111.76 74.93)
 		)
 		(stroke
@@
 	(wire
 		(pts
-			(xy 121.92 44.45) (xy 121.92 72.39)
+			(xy 124.46 44.45) (xy 124.46 72.39)
 		)
 		(stroke
@@
 	(wire
 		(pts
-			(xy 121.92 44.45) (xy 97.79 44.45)
+			(xy 124.46 44.45) (xy 97.79 44.45)
+		)
+		(stroke
+			(width 0)
+			(type default)
+		)
+	)
+	(wire
+		(pts
+			(xy 104.14 55.88) (xy 111.76 55.88)
 		)
 		(stroke
@@
 	(wire
 		(pts
-			(xy 104.14 52.07) (xy 119.38 52.07)
-		)
-		(stroke
-			(width 0)
-			(type default)
-		)
-	)
-	(wire
-		(pts
 			(xy 199.39 62.23) (xy 203.2 62.23)
 		)
@@
 	(wire
 		(pts
-			(xy 104.14 67.31) (xy 104.14 71.12)
+			(xy 104.14 55.88) (xy 104.14 71.12)
 		)
 		(stroke
@@
 		(pts
 			(xy 167.64 57.15) (xy 171.45 57.15)
+		)
+		(stroke
+			(width 0)
+			(type default)
+		)
+	)
+	(wire
+		(pts
+			(xy 111.76 74.93) (xy 132.08 74.93)
 		)
 		(stroke
@@
 		)
 	)
-	(global_label "HP.ENG.IGN.ALM"
+	(global_label "HP.IGN.75.TRL.SBY.A"
 		(shape input)
 		(at 52.07 71.12 180)
@@
 		)
 	)
-	(global_label "HP.ENG.IGN.SBY"
+	(global_label "HP.IGN.75.TRL.SBY.B"
 		(shape input)
 		(at 52.07 74.93 180)
@@
 	(symbol
 		(lib_id "Device:LED")
-		(at 104.14 58.42 270)
+		(at 111.76 62.23 270)
 		(unit 1)
 		(exclude_from_sim no)
@@
 		(dnp no)
 		(property "Reference" "D1"
-			(at 100.838 57.912 90)
+			(at 108.458 61.722 90)
 			(effects
 				(font
@@
 		)
 		(property "Value" "ALARM"
-			(at 109.22 57.912 90)
+			(at 116.84 61.722 90)
 			(effects
 				(font
@@
 		)
 		(property "Footprint" ""
-			(at 104.14 58.42 0)
+			(at 111.76 62.23 0)
 			(effects
 				(font
@@
 		)
 		(property "Datasheet" "~"
-			(at 104.14 58.42 0)
+			(at 111.76 62.23 0)
 			(effects
 				(font
@@
 		)
 		(property "Description" ""
-			(at 104.14 58.42 0)
+			(at 111.76 62.23 0)
 			(effects
 				(font
@@
 	(symbol
 		(lib_id "Device:R_Small")
-		(at 104.14 64.77 0)
+		(at 111.76 68.58 0)
 		(unit 1)
 		(exclude_from_sim no)
@@
 		(dnp no)
 		(property "Reference" "R1"
-			(at 100.838 64.516 0)
+			(at 108.458 68.326 0)
 			(effects
 				(font
@@
 		)
 		(property "Value" "R_Small"
-			(at 106.68 66.0399 0)
+			(at 114.3 69.8499 0)
 			(effects
 				(font
@@
 		)
 		(property "Footprint" ""
-			(at 104.14 64.77 0)
+			(at 111.76 68.58 0)
 			(effects
 				(font
@@
 		)
 		(property "Datasheet" "~"
-			(at 104.14 64.77 0)
+			(at 111.76 68.58 0)
 			(effects
 				(font
@@
 		)
 		(property "Description" "Resistor, small symbol"
-			(at 104.14 64.77 0)
-			(effects
-				(font
+			(at 111.76 68.58 0)
+			(effects
+				(font
