File: resources/kicad/schematics/dc/helm/helm-switches.kicad_sch (KiCad schematic)
At the start: 46 parts, among them SW01 CARLING_TYPE_21_OFF-ON, SW02 CARLING_TYPE_28_(ON)-OFF-(ON), SW03 CARLING_TYPE_22_OFF-(ON), SW04 CARLING_TYPE_62_OFF-ON-ON, SW05 CARLING_TYPE_21_OFF-ON, SW06 CARLING_BLANK, SW07 CARLING_BLANK, SW08 CARLING_BLANK, SW09 CARLING_TYPE_21_OFF-ON, SW10 CARLING_TYPE_21_OFF-ON, SW11 CARLING_TYPE_21_OFF-ON, SW12 CARLING_TYPE_21_OFF-ON, SW13 CARLING_TYPE_21_OFF-ON, SW14 CARLING_TYPE_21_OFF-ON, SW15 CARLING_TYPE_21_OFF-ON, SW16 CARLING_TYPE_62_OFF-ON-ON, SW17 CARLING_TYPE_24_ON-ON, SW18 CARLING_TYPE_22_OFF-(ON), SW19 CARLING_TYPE_62_OFF-ON-ON, SW20 CARLING_TYPE_62_OFF-ON-ON, SW21 CARLING_TYPE_62_OFF-ON-ON, SW22 CARLING_TYPE_62_OFF-ON-ON, SW23 CARLING_BLANK, SW24 CARLING_TYPE_62_OFF-ON-ON, SW25 CARLING_TYPE_21_OFF-ON, SW26 CARLING_V_SERIES_ROTARY_TYPE_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, SW27 CARLING_TYPE_62_OFF-ON-ON, SW28 CARLING_TYPE_28_(ON)-OFF-(ON), SW29 CARLING_TYPE_28_(ON)-OFF-(ON), SW30 CARLING_TYPE_28_(ON)-OFF-(ON), SW31 CARLING_TYPE_62_OFF-ON-ON, SW32 CARLING_TYPE_62_OFF-ON-ON, SW33 CARLING_BLANK, SW34 CARLING_BLANK, SW35 CARLING_BLANK, SW36 CARLING_TYPE_62_OFF-ON-ON, SW37 CARLING_TYPE_21_OFF-ON, SW38 CARLING_TYPE_21_OFF-ON, SW39 CARLING_TYPE_26_ON-OFF-ON

Commit message: Tweak
Parts:
- SW01: value CARLING_TYPE_21_OFF-ON -> ILLUM
- SW02: value CARLING_TYPE_28_(ON)-OFF-(ON) -> PANEL
- SW03: value CARLING_TYPE_22_OFF-(ON) -> SILENCE
Changed lines of the file:
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@@
 	)
 	(symbol
+		(lib_name "Carling_L_Series_Type_28_(ON)-OFF-(ON)_1")
 		(lib_id "Switch:Carling_L_Series_Type_28_(ON)-OFF-(ON)")
 		(at 144.78 39.37 0)
@@
 		(dnp no)
 		(property "Reference" "SW02"
-			(at 144.78 27.686 0)
-			(effects
-				(font
-					(size 1.27 1.27)
-				)
-			)
-		)
-		(property "Value" "CARLING_TYPE_28_(ON)-OFF-(ON)"
-			(at 144.78 51.308 0)
+			(at 139.446 27.686 0)
+			(effects
+				(font
+					(size 1.27 1.27)
+				)
+			)
+		)
+		(property "Value" "PANEL"
+			(at 149.606 27.686 0)
 			(effects
 				(font
@@
 			)
 		)
-		(property "Description" ""
-			(at 126.492 26.416 0)
-			(effects
-				(font
-					(size 1.27 1.27)
-				)
-				(hide yes)
+		(property "Description" "Type 28, (ON)-OFF-(ON)"
+			(at 144.78 51.054 0)
+			(effects
+				(font
+					(size 1.27 1.27)
+				)
 			)
 		)
@@
 		(dnp no)
 		(property "Reference" "SW01"
-			(at 101.6 27.686 0)
-			(effects
-				(font
-					(size 1.27 1.27)
-				)
-			)
-		)
-		(property "Value" "CARLING_TYPE_21_OFF-ON"
-			(at 101.6 51.308 0)
+			(at 96.52 27.686 0)
+			(effects
+				(font
+					(size 1.27 1.27)
+				)
+			)
+		)
+		(property "Value" "ILLUM"
+			(at 106.68 27.686 0)
 			(effects
 				(font
@@
 			)
 		)
-		(property "Description" ""
-			(at 83.312 26.416 0)
-			(effects
-				(font
-					(size 1.27 1.27)
-				)
-				(hide yes)
+		(property "Description" "Type 21, OFF-ON"
+			(at 101.6 51.054 0)
+			(effects
+				(font
+					(size 1.27 1.27)
+				)
 			)
 		)
@@
 	)
 	(symbol
+		(lib_name "Carling_L_Series_Type_22_OFF-(ON)_1")
 		(lib_id "Switch:Carling_L_Series_Type_22_OFF-(ON)")
 		(at 187.96 39.37 0)
@@
 		(dnp no)
 		(property "Reference" "SW03"
-			(at 187.96 27.686 0)
-			(effects
-				(font
-					(size 1.27 1.27)
-				)
-			)
-		)
-		(property "Value" "CARLING_TYPE_22_OFF-(ON)"
-			(at 187.96 51.308 0)
+			(at 182.88 27.686 0)
+			(effects
+				(font
+					(size 1.27 1.27)
+				)
+			)
+		)
+		(property "Value" "SILENCE"
+			(at 191.77 27.686 0)
 			(effects
 				(font
@@
 			)
 		)
-		(property "Description" ""
-			(at 169.672 26.416 0)
-			(effects
-				(font
-					(size 1.27 1.27)
-				)
-				(hide yes)
-			)
-		)
+		(property "Description" "Type 22, OFF-(ON)"
+			(at 187.96 51.054 0)
+			(effects
+				(font
+					(size 1.27 1.27)
+				)
+			)
+		)

Commit message: Many tweaks
Parts:
- removed SW01: ILLUM, symbol Switch:Carling_L_Series_Type_21_OFF-ON
- removed SW04, SW31, SW32: CARLING_TYPE_62_OFF-ON-ON, symbol Switch:Carling_L_Series_Type_62_OFF-ON-ON
- removed SW10, SW11, SW12, SW13, SW14, SW15, SW25, SW37, SW38: CARLING_TYPE_21_OFF-ON, symbol Switch:Carling_L_Series_Type_21_OFF-ON
- removed SW39: CARLING_TYPE_26_ON-OFF-ON, symbol Switch:Carling_L_Series_Type_26_ON-OFF-ON
- added F1: 5A, symbol Device:Fuse
- added SW01: ILLUM, symbol Switch:Carling_L_Series_Type_68_ON-ON-ON
- added SW04: WASTE, symbol Switch:Carling_L_Series_Type_68_ON-ON-ON
- added SW10: NAV, symbol Switch:Carling_L_Series_Type_24_ON-ON
- added SW11: ANCHOR, symbol Switch:Carling_L_Series_Type_24_ON-ON
- added SW12: WORK, symbol Switch:Carling_L_Series_Type_24_ON-ON
- added SW13: SRCH, symbol Switch:Carling_L_Series_Type_24_ON-ON
- added SW14: DECK, symbol Switch:Carling_L_Series_Type_24_ON-ON
- added SW15: NIGHT, symbol Switch:Carling_L_Series_Type_24_ON-ON
- added SW25: POWER, symbol Switch:Carling_L_Series_Type_68_ON-ON-ON
- added SW31: AIS, symbol Switch:Carling_L_Series_Type_68_ON-ON-ON
- added SW32: WIFI, symbol Switch:Carling_L_Series_Type_24_ON-ON
- added SW37: TROLL, symbol Switch:Carling_L_Series_Type_24_ON-ON
- added SW38: SPUD, symbol Switch:Carling_L_Series_Type_28_(ON)-OFF-(ON)
- added SW39: UP-DN, symbol Switch:Carling_L_Series_Type_72_ON-OFF-ON
- SW05: value CARLING_TYPE_21_OFF-ON -> DWASH
- SW09: value CARLING_TYPE_21_OFF-ON -> FLUSH
- SW16: value CARLING_TYPE_62_OFF-ON-ON -> WIPER
- SW17: value CARLING_TYPE_24_ON-ON -> BOARD
- SW18: value CARLING_TYPE_22_OFF-(ON) -> HORN
- SW19, SW21: value CARLING_TYPE_62_OFF-ON-ON -> EROOM
- SW20, SW22: value CARLING_TYPE_62_OFF-ON-ON -> MCOMP
- SW24: value CARLING_TYPE_62_OFF-ON-ON -> CRTSY
- SW26: value CARLING_V_SERIES_ROTARY_TYPE_26_ON-OFF-ON -> ~
- SW27: value CARLING_TYPE_62_OFF-ON-ON -> ENABLE
- SW28: value CARLING_TYPE_28_(ON)-OFF-(ON) -> HATCH
- SW29: value CARLING_TYPE_28_(ON)-OFF-(ON) -> MAST
- SW30: value CARLING_TYPE_28_(ON)-OFF-(ON) -> ANCHOR
- SW36: value CARLING_TYPE_62_OFF-ON-ON -> RADAR
Connections:
- net F5.1.6.HPA.RST: now also SW03.6; no longer SW03.4
- net F5.1.7: now also SW02.6, SW01.8
- net F5.1.7.HPD.DEC: now also SW02.8; no longer SW02.4
- net F5.1.7.HPD.INC: now also SW02.5; no longer SW02.1
- net F5.1.7.HPD.SBY: now also SW01.7
- net F9.1.11: now also SW18.8; no longer SW18.2
- net F9.1.11.HRN.OP1: now also SW18.6; no longer SW18.4
- net F9.1.2: now also SW03.8, SW05.8, SW09.8, SW04.4, SW04.8, SW31.12 (LED+), SW32.11 (LED-), SW32.9 (LED-); no longer SW02.10 (LED+), SW02.2, SW03.10 (LED+), SW05.10 (LED+), SW05.12 (LED+), SW05.2, SW09.10 (LED+), SW09.12 (LED+), SW09.2
- net F9.1.2.DSP.OP1: now also SW04.7
- net F9.1.2.DSP.SBY: now also SW04.2
- net F9.1.2.DWP.OP1: now also SW05.6; no longer SW05.4
- net F9.1.2.TFP.OP1: now also SW09.6; no longer SW09.4
- net F9.1.3: now also SW31.4, SW31.8
- net F9.1.3.AIS.OP2: now also SW31.7
- net F9.1.3.AIS.SBY: now also SW31.10 (LED+), SW31.2
- net F9.1.7: now also SW32.6
- net F9.1.7.WIF.OP1: now also SW32.7
- net F9.1.7.WIF.OP2: now also SW32.5
- net F9.1.8: now also SW38.4, SW38.5
- net F9.2.1: now also SW27.10 (LED+), SW27.3, SW10.8, SW11.8, SW12.8, SW13.8, SW14.8, SW15.8, SW25.10 (LED+), SW38.10 (LED+); no longer SW16.10 (LED+), SW16.12 (LED+), SW17.10 (LED+), SW18.10 (LED+)
- net F9.2.3.BBD.A: no longer SW17.12 (LED+)
- net F9.2.7: no longer SW16.3
- net F9.2.7.WPR.CFG: no longer SW16.2
- net F9.2.7.WPR.OP1: no longer SW16.4
- net F9.2.8.THR.ACT: now also SW25.2, SW25.7; no longer SW27.3
- net F9.2.8.THR.OP1: now also SW25.12 (LED+), SW25.4; no longer SW27.2
- net F9.2.8.THR.OP2: now also SW25.8; no longer SW27.4
- net GND: now also SW16.9 (LED-), SW17.9 (LED-), SW18.9 (LED-), SW10.9 (LED-), SW11.9 (LED-), SW12.9 (LED-), SW13.9 (LED-), SW14.9 (LED-), SW15.9 (LED-), SW38.1, SW38.7
- net GND.HPD.PWM: now also SW24.6, SW28.5, SW28.8, SW29.5, SW29.8, SW30.5, SW30.8, SW36.8, SW25.9 (LED-), SW31.9 (LED-), SW32.1, SW32.12 (LED+), SW37.6, SW37.9 (LED-), SW38.9 (LED-), SW39.9 (LED-); no longer SW02.9 (LED-), SW03.9 (LED-), SW05.6, SW05.9 (LED-), SW09.6, SW09.9 (LED-), SW16.6, SW16.9 (LED-), SW17.11 (LED-), SW17.9 (LED-), SW18.9 (LED-), SW27.6, SW36.6
- net GND.HPD.PWM.INT: now also SW25.11 (LED-); no longer SW24.6, SW27.8, SW36.8
- net GND.HPD.PWN.INT: now also IN6.10 (LED+), IN6.12 (LED+); no longer IN6.11 (LED-), IN6.9 (LED-)
- net HPA.10: now also IN6.11 (LED-); no longer IN6.12 (LED+)
- net HPA.9: now also IN6.9 (LED-); no longer IN6.10 (LED+)
- net IGN.75: now also F1.2
- net IGN.75.TRL.SBY: now also SW37.1
- net at SW05.11 (LED-): no longer SW05.8
- net at SW27.12 (LED+), SW28.10 (LED+), SW28.2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: now also SW27.2, SW27.4, SW28.12 (LED+), SW29.12 (LED+), SW30.12 (LED+); no longer SW26.8 (LED+), SW27.10 (LED+)
- net at SW27.11 (LED-): no longer SW27.7
- net HPD.SBY.PWM: now reaches SW02.12 (LED+)
- net HPD.SBY.PWM: now also SW03.12 (LED+), SW05.12 (LED+), SW05.4, SW09.12 (LED+), SW09.4, SW16.12 (LED+), SW17.12 (LED+), SW18.12 (LED+), SW01.12 (LED+), SW01.4, SW04.12 (LED+), SW10.12 (LED+), SW10.4, SW11.12 (LED+), SW11.4, SW12.12 (LED+), SW12.4, SW13.12 (LED+), SW13.4, SW14.12 (LED+), SW14.4, SW15.12 (LED+), SW15.4
- net at SW29.11 (LED-): now also SW29.6
- net at SW28.11 (LED-): now also SW28.6
- net at SW30.11 (LED-): now also SW30.6
- net at SW16.11 (LED-): no longer SW16.7
- net at SW09.11 (LED-): no longer SW09.8
- net F5.1.6: no longer names the net of SW03.2
- new net: F1.1, SW37.10 (LED+), SW37.12 (LED+), SW37.2
- new net: SW12.10 (LED+), SW12.2
- new net: SW05.10 (LED+), SW05.2
- new net: SW14.10 (LED+), SW14.2
- new net: SW13.10 (LED+), SW13.2
- new net: SW37.11 (LED-), SW37.8
- new net: SW01.10 (LED+), SW01.2
- new net: SW32.10 (LED+), SW32.2
- new net: SW10.10 (LED+), SW10.2
- new net: SW39.10 (LED+), SW39.5
- new net: SW39.12 (LED+), SW39.4
- new net: SW11.10 (LED+), SW11.2
- new net: SW15.10 (LED+), SW15.2
- new net: SW09.10 (LED+), SW09.2
- new net F9.1.8.A: SW38.6
- new net F9.1.8.B: SW38.2
- new net F9.2.1.DKL: SW14.6
- new net GND.ANL: SW11.6
- new net GND.NVL: SW10.6
- new net GND.SRL: SW13.6
- new net GND.WKL: SW12.6
- new net GND.WNL: SW15.6
- new net HP.GND: SW01.9 (LED-), SW02.9 (LED-), SW03.9 (LED-), SW04.9 (LED-), SW05.9 (LED-), SW09.9 (LED-)
- new net SP.DN: SW39.8
- new net SP.POS: SW38.12 (LED+), SW39.2, SW39.7
- new net SP.UP: SW39.1

Commit message: Swap dimmer polarity
Parts:
- removed SW19, SW21: EROOM, symbol Switch:Carling_L_Series_Type_62_OFF-ON-ON
- removed SW20, SW22: MCOMP, symbol Switch:Carling_L_Series_Type_62_OFF-ON-ON
- removed SW24: CRTSY, symbol Switch:Carling_L_Series_Type_62_OFF-ON-ON
- added SW19, SW21: EROOM, symbol Switch:Carling_L_Series_Type_68_ON-ON-ON
- added SW20, SW22: MCOMP, symbol Switch:Carling_L_Series_Type_68_ON-ON-ON
- added SW24: CRTSY, symbol Switch:Carling_L_Series_Type_24_ON-ON
Connections:
- net F5.1.4: now also SW19.4, SW19.8
- net F5.1.4.EBP.OP1: now also SW19.7
- net F5.1.4.EBP.SBY: now also SW19.2
- net F5.1.5: now also SW20.4, SW20.8
- net F5.1.5.MBP.OP1: now also SW20.7
- net F5.1.5.MBP.SBY: now also SW20.2
- net F9.1.2: now also SW21.4, SW21.8, SW22.4, SW22.8
- net F9.1.2.ERV.OP1: now also SW21.7
- net F9.1.2.ERV.SBY: now also SW21.2
- net F9.1.2.MBV.OP1: now also SW22.7
- net F9.1.2.MBV.SBY: now also SW22.2
- net GND: now also SW19.9 (LED-), SW20.9 (LED-), SW21.9 (LED-), SW22.9 (LED-), SW24.8, SW24.9 (LED-)
- net GND.CTL.OP1: now also SW24.6
- net HPD.SBY.PWM: now also SW19.12 (LED+), SW20.12 (LED+), SW21.12 (LED+), SW22.12 (LED+), SW24.12 (LED+), SW24.4
- new net: SW24.10 (LED+), SW24.2
